Commit message: updated urdf and config files

File: mobo_bot_description/urdf/part_macros.xacro (robot description, xacro)
@@ -1,10 +1,10 @@
 <?xml version="1.0"?>
 <robot name="mobo_bot" xmlns:xacro="http://www.ros.org/wiki/xacro" >
-    <xacro:macro name="box_with_fillet" params="size_x size_y size_z fr material x y z">
+    <xacro:macro name="box_with_fillet" params="x y z size_x size_y size_z fillet_radius material">
             <!-- logitudinal box -->
             <visual>
                 <origin xyz="${x} ${y} ${z}" rpy="0 0 0"/>
                 <geometry>
-                    <box size="${size_x} ${size_y-(2*fr)} ${size_z}"/>
+                    <box size="${size_x} ${size_y-(2*fillet_radius)} ${size_z}"/>
                 </geometry>
                 <material name="${material}"/>
@@ -14,5 +14,5 @@
                 <origin xyz="${x} ${y} ${z}" rpy="0 0 0"/>
                 <geometry>
-                    <box size="${size_x-(2*fr)} ${size_y} ${size_z}"/>
+                    <box size="${size_x-(2*fillet_radius)} ${size_y} ${size_z}"/>
                 </geometry>
                 <material name="${material}"/>
@@ -20,7 +20,7 @@
             <!-- cylinder1 -->
             <visual>
-                <origin xyz="${x+((size_x/2)-fr)} ${y+((size_y/2)-fr)} ${z}" rpy="0 0 0"/>
+                <origin xyz="${x+((size_x/2)-fillet_radius)} ${y+((size_y/2)-fillet_radius)} ${z}" rpy="0 0 0"/>
                 <geometry>
-                    <cylinder length="${size_z}" radius="${fr}"/>
+                    <cylinder length="${size_z}" radius="${fillet_radius}"/>
                 </geometry>
                 <material name="${material}"/>
@@ -28,7 +28,7 @@
             <!-- cylinder2 -->
             <visual>
-                <origin xyz="${x+((size_x/2)-fr)} ${y-((size_y/2)-fr)} ${z}" rpy="0 0 0"/>
+                <origin xyz="${x+((size_x/2)-fillet_radius)} ${y-((size_y/2)-fillet_radius)} ${z}" rpy="0 0 0"/>
                 <geometry>
-                    <cylinder length="${size_z}" radius="${fr}"/>
+                    <cylinder length="${size_z}" radius="${fillet_radius}"/>
                 </geometry>
                 <material name="${material}"/>
@@ -36,7 +36,7 @@
             <!-- cylinder3 -->
             <visual>
-                <origin xyz="${x-((size_x/2)-fr)} ${y+((size_y/2)-fr)} ${z}" rpy="0 0 0"/>
+                <origin xyz="${x-((size_x/2)-fillet_radius)} ${y+((size_y/2)-fillet_radius)} ${z}" rpy="0 0 0"/>
                 <geometry>
-                    <cylinder length="${size_z}" radius="${fr}"/>
+                    <cylinder length="${size_z}" radius="${fillet_radius}"/>
                 </geometry>
                 <material name="${material}"/>
@@ -44,10 +44,63 @@
             <!-- cylinder4 -->
             <visual>
-                <origin xyz="${x-((size_x/2)-fr)} ${y-((size_y/2)-fr)} ${z}" rpy="0 0 0"/>
+                <origin xyz="${x-((size_x/2)-fillet_radius)} ${y-((size_y/2)-fillet_radius)} ${z}" rpy="0 0 0"/>
                 <geometry>
-                    <cylinder length="${size_z}" radius="${fr}"/>
+                    <cylinder length="${size_z}" radius="${fillet_radius}"/>
                 </geometry>
                 <material name="${material}"/>
             </visual>
     </xacro:macro>
+    <xacro:property name="wheel_radius" value="0.05"/>
+    <xacro:property name="wheel_width" value="0.04"/>
+    <xacro:property name="wheel_mass" value="0.5"/>
+    <xacro:property name="wheel_color" value="black"/>
+    <xacro:property name="rim_color" value="red"/>
+   <xacro:macro name="insert_drive_wheel">
+        <visual>
+            <origin xyz="0 0 0" rpy="0 0 0"/>
+            <geometry>
+                <cylinder radius="${wheel_radius}" length="${wheel_width}"/>
+            </geometry>
+            <material name="${wheel_color}"/>
+        </visual>
+        <collision>
+           <origin xyz="0 0 0" rpy="0 0 0"/>
+            <geometry>
+                <cylinder radius="${wheel_radius}" length="${wheel_width}"/>
+            </geometry>
+        </collision>
+        <xacro:inertial_cylinder mass="${wheel_mass}" length="${wheel_width}" radius="${wheel_radius}">
+            <origin xyz="0 0 0" rpy="0 0 0"/>
+        </xacro:inertial_cylinder>
+    </xacro:macro>
+    <xacro:macro name="insert_wheel_rim">
+        <visual>
+            <origin xyz="0 0 0" rpy="0 0 0"/>
+            <geometry>
+                <box size="0.01 ${wheel_radius*1.2} ${wheel_width+0.005}"/>
+            </geometry>
+            <material name="${rim_color}"/>
+        </visual>
+        <visual>
+            <origin xyz="0 0 0" rpy="0 0 ${pi/2}"/>
+            <geometry>
+                <box size="0.01 ${wheel_radius*1.2} ${wheel_width+0.005}"/>
+            </geometry>
+            <material name="${rim_color}"/>
+        </visual>
+        <visual>
+            <origin xyz="0 0 0" rpy="0 0 ${-pi/4}"/>
+            <geometry>
+                <box size="0.01 ${wheel_radius*1.2} ${wheel_width+0.005}"/>
+            </geometry>
+            <material name="${rim_color}"/>
+        </visual>
+        <visual>
+            <origin xyz="0 0 0" rpy="0 0 ${pi/4}"/>
+            <geometry>
+                <box size="0.01 ${wheel_radius*1.2} ${wheel_width+0.005}"/>
+            </geometry>
+            <material name="${rim_color}"/>
+        </visual>
+    </xacro:macro>
 </robot>

File: mobo_bot_description/urdf/robot_urdf_description.xacro (robot description, xacro)
@@ -9,5 +9,17 @@
     <xacro:arg name="imu_visual"   default="true"/>
     <xacro:arg name="sonar_visual"   default="false"/>
-    <xacro:arg name="cam_visual"   default="true"/>
+    <xacro:arg name="cam_visual"   default="false"/>
+     <!-- GAZEBO WHEEL PARAMETERS -->
+    <xacro:macro name="gazebo_wheel_settings" params="name">
+        <gazebo reference="${name}">
+            <mu1>1.0</mu1>
+            <mu2>1.0</mu2>
+            <!-- <kp>${kp}</kp> -->
+            <!-- <kd>${kd}</kd> -->
+            <!-- <fdir1>${fdir}</fdir1> -->
+            <!-- <minDepth>${minDepth}</minDepth> -->
+            <material>Gazebo/FlatBlack</material>
+        </gazebo>
+    </xacro:macro>
     <!-- BASE LINK -->
     <!-- <base joint/> -->
@@ -22,5 +34,5 @@
     </joint>
     <link name="base_chassis_link">
-        <xacro:box_with_fillet size_x="0.4" size_y="0.30" size_z="${base_chassis_height}" fr="0.1" material="white" x="-0.06" y="0" z="${base_chassis_height/2}"/>
+        <xacro:box_with_fillet x="-0.06" y="0" z="${base_chassis_height/2}" size_x="0.4" size_y="0.30" size_z="${base_chassis_height}" fillet_radius="0.1" material="white"/>
         <collision>
            <origin xyz="-0.06 0 ${base_chassis_height/2}" rpy="0 0 0"/>
@@ -45,30 +57,7 @@
     </joint>
     <link name="left_wheel_link">
-        <visual>
-            <origin xyz="0 0 0" rpy="0 0 0"/>
-            <geometry>
-                <cylinder radius="0.05" length="0.04"/>
-            </geometry>
-            <material name="black"/>
-        </visual>
-        <collision>
-           <origin xyz="0 0 0" rpy="0 0 0"/>
-            <geometry>
-                <sphere radius="0.05" />
-            </geometry>
-        </collision>
-        <xacro:inertial_cylinder mass="0.5" length="0.04" radius="0.05">
-            <origin xyz="0 0 0" rpy="0 0 0"/>
-        </xacro:inertial_cylinder>
+        <xacro:insert_drive_wheel/>
     </link>
-    <gazebo reference="left_wheel_link">
-        <mu1>1.0</mu1>
-        <mu2>1.0</mu2>
-        <!-- <kp>1000000.0</kp>
-        <kd>1.0</kd>
-        <fdir1>1 0 0</fdir1>
-        <minDepth>0.1</minDepth> -->
-        <material>Gazebo/FlatBlack</material>
-    </gazebo>
+    <xacro:gazebo_wheel_settings name="left_wheel_link"/>
     <joint name="left_wheel_rim_joint" type="fixed">
         <parent link="left_wheel_link"/>
@@ -77,32 +66,5 @@
     </joint>
     <link name="left_wheel_rim_link">
-        <visual>
-            <origin xyz="0 0 0" rpy="0 0 0"/>
-            <geometry>
-                <box size="0.01 0.06 0.0405"/>
-            </geometry>
-            <material name="red"/>
-        </visual>
-        <visual>
-            <origin xyz="0 0 0" rpy="0 0 ${pi/2}"/>
-            <geometry>
-                <box size="0.01 0.06 0.0405"/>
-            </geometry>
-            <material name="red"/>
-        </visual>
-        <visual>
-            <origin xyz="0 0 0" rpy="0 0 ${-pi/4}"/>
-            <geometry>
-                <box size="0.01 0.06 0.0405"/>
-            </geometry>
-            <material name="red"/>
-        </visual>
-        <visual>
-            <origin xyz="0 0 0" rpy="0 0 ${pi/4}"/>
-            <geometry>
-                <box size="0.01 0.06 0.0405"/>
-            </geometry>
-            <material name="red"/>
-        </visual>
+        <xacro:insert_wheel_rim/>
     </link>
     <gazebo reference="left_wheel_rim_link">
@@ -118,30 +80,7 @@
     </joint>
     <link name="right_wheel_link">
-        <visual>
-            <origin xyz="0 0 0" rpy="0 0 0"/>
-            <geometry>
-                <cylinder radius="0.05" length="0.04"/>
-            </geometry>
-            <material name="black"/>
-        </visual>
-        <collision>
-           <origin xyz="0 0 0" rpy="0 0 0"/>
-            <geometry>
-                <sphere radius="0.05" />
-            </geometry>
-        </collision>
-        <xacro:inertial_cylinder mass="0.5" length="0.04" radius="0.05">
-            <origin xyz="0 0 0" rpy="0 0 0"/>
-        </xacro:inertial_cylinder>
+        <xacro:insert_drive_wheel/>
     </link>
-    <gazebo reference="right_wheel_link">
-        <mu1>1.0</mu1>
-        <mu2>1.0</mu2>
-        <!-- <kp>1000000.0</kp>
-        <kd>1.0</kd>
-        <fdir1>1 0 0</fdir1>
-        <minDepth>0.1</minDepth> -->
-        <material>Gazebo/FlatBlack</material>
-    </gazebo>
+    <xacro:gazebo_wheel_settings name="right_wheel_link"/>
     <joint name="right_wheel_rim_joint" type="fixed">
         <parent link="right_wheel_link"/>
@@ -150,37 +89,9 @@
     </joint>
     <link name="right_wheel_rim_link">
-        <visual>
-            <origin xyz="0 0 0" rpy="0 0 0"/>
-            <geometry>
-                <box size="0.01 0.06 0.0405"/>
-            </geometry>
-            <material name="red"/>
-        </visual>
-        <visual>
-            <origin xyz="0 0 0" rpy="0 0 ${pi/2}"/>
-            <geometry>
-                <box size="0.01 0.06 0.0405"/>
-            </geometry>
-            <material name="red"/>
-        </visual>
-        <visual>
-            <origin xyz="0 0 0" rpy="0 0 ${-pi/4}"/>
-            <geometry>
-                <box size="0.01 0.06 0.0405"/>
-            </geometry>
-            <material name="red"/>
-        </visual>
-        <visual>
-            <origin xyz="0 0 0" rpy="0 0 ${pi/4}"/>
-            <geometry>
-                <box size="0.01 0.06 0.0405"/>
-            </geometry>
-            <material name="red"/>
-        </visual>
+        <xacro:insert_wheel_rim/>
     </link>
     <gazebo reference="right_wheel_rim_link">
         <material>Gazebo/Red</material>
     </gazebo>
-    <!--  ########################### -->
     <!--  CASTER WHEEL LINK -->
     <joint name="caster_wheel_joint" type="fixed">

Commit message: update robot code

File: mobo_bot_description/urdf/part_macros.xacro (robot description, xacro)
@@ -50,4 +50,27 @@
                 <material name="${material}"/>
             </visual>
+    </xacro:macro>
+    <xacro:macro name="insert_mesh_drive_wheel">
+        <visual>
+            <origin xyz="0 0 0" rpy="0 0 0"/>
+            <geometry>
+                <xacro:unless value="${gazebo_visual}">
+                    <mesh filename="package://mobo_bot_description/meshes/wheel.stl"/>
+                </xacro:unless>
+                <xacro:if value="${gazebo_visual}">
+                    <mesh filename="$(find mobo_bot_description)/meshes/wheel.stl"/>
+                </xacro:if>
+            </geometry>
+            <material name="black"/>
+        </visual>
+        <collision>
+            <origin xyz="0 0 0" rpy="0 0 0"/>
+            <geometry>
+                <cylinder radius="0.05" length="0.02"/>
+            </geometry>
+        </collision>
+        <xacro:inertial_cylinder mass="0.4" length="0.02" radius="0.05">
+            <origin xyz="0 0 0" rpy="0 0 0"/>
+        </xacro:inertial_cylinder>
     </xacro:macro>
     <xacro:property name="wheel_radius" value="0.05"/>
@@ -104,3 +127,14 @@
         </visual>
     </xacro:macro>
+    <!-- <joint name="right_wheel_rim_joint" type="fixed">
+        <parent link="right_wheel_link"/>
+        <child link="right_wheel_rim_link"/>
+        <origin xyz="0 0 0" rpy="0 0 0"/>
+    </joint>
+    <link name="right_wheel_rim_link">
+        <xacro:insert_wheel_rim/>
+    </link>
+    <gazebo reference="right_wheel_rim_link">
+        <material>Gazebo/Red</material>
+    </gazebo> -->
 </robot>

File: mobo_bot_description/urdf/robot_urdf_description.xacro (robot description, xacro)
@@ -4,6 +4,7 @@
     <xacro:include filename="$(find mobo_bot_description)/urdf/part_macros.xacro"/>
     <xacro:include filename="$(find mobo_bot_description)/urdf/inertia_macros.xacro"/>
+    <xacro:property name="gazebo_visual" value="true"/>
     <xacro:property name="use_ros2_control" value="false"/>
-    <xacro:property name="base_chassis_height" value="0.1"/>
+    <xacro:property name="base_chassis_height" value="0.15"/>
     <xacro:arg name="laser_visual" default="false"/>
     <xacro:arg name="imu_visual"   default="true"/>
@@ -18,5 +19,5 @@
             <!-- <kd>${kd}</kd> -->
             <!-- <fdir1>${fdir}</fdir1> -->
-            <!-- <minDepth>${minDepth}</minDepth> -->
+            <minDepth>0.01</minDepth>
             <material>Gazebo/FlatBlack</material>
         </gazebo>
@@ -27,4 +28,11 @@
     </link>
     <!-- ################# -->
+    <joint name="base_footprint_joint" type="fixed">
+        <parent link="base_link"/>
+        <child link="base_footprint"/>
+        <origin xyz="0 0 0" rpy="0 0 0"/>
+    </joint>
+    <link name="base_footprint">
+    </link>
     <!-- CHASSIS LINK -->
     <joint name="base_chassis_joint" type="fixed">
@@ -34,13 +42,13 @@
     </joint>
     <link name="base_chassis_link">
-        <xacro:box_with_fillet x="-0.06" y="0" z="${base_chassis_height/2}" size_x="0.4" size_y="0.30" size_z="${base_chassis_height}" fillet_radius="0.1" material="white"/>
+        <xacro:box_with_fillet x="-0.05" y="0" z="${base_chassis_height/2}" size_x="0.4" size_y="0.37" size_z="${base_chassis_height}" fillet_radius="0.1" material="white"/>
         <collision>
-           <origin xyz="-0.06 0 ${base_chassis_height/2}" rpy="0 0 0"/>
+           <origin xyz="-0.05 0 ${base_chassis_height/2}" rpy="0 0 0"/>
             <geometry>
-                <box size="0.4 0.29 ${base_chassis_height}"/>
+                <box size="0.4 0.37 ${base_chassis_height}"/>
             </geometry>
         </collision>
-        <xacro:inertial_box mass="5.0" x="0.4" y="0.30" z="${base_chassis_height}">
-            <origin xyz="-0.06 0 ${base_chassis_height/2}" rpy="0 0 0"/>
+        <xacro:inertial_box mass="5.0" x="0.4" y="0.37" z="${base_chassis_height}">
+            <origin xyz="-0.05 0 ${base_chassis_height/2}" rpy="0 0 0"/>
         </xacro:inertial_box>
     </link>
@@ -53,22 +61,11 @@
         <parent link="base_chassis_link"/>
         <child link="left_wheel_link"/>
-        <origin xyz="0 0.17 0" rpy="${-pi/2} 0 0"/>
+        <origin xyz="0 0.2 0" rpy="${-pi/2} 0 0"/>
         <axis xyz="0 0 1"/>
     </joint>
     <link name="left_wheel_link">
-        <xacro:insert_drive_wheel/>
+        <xacro:insert_mesh_drive_wheel/>
     </link>
     <xacro:gazebo_wheel_settings name="left_wheel_link"/>
-    <joint name="left_wheel_rim_joint" type="fixed">
-        <parent link="left_wheel_link"/>
-        <child link="left_wheel_rim_link"/>
-        <origin xyz="0 0 0" rpy="0 0 0"/>
-    </joint>
-    <link name="left_wheel_rim_link">
-        <xacro:insert_wheel_rim/>
-    </link>
-    <gazebo reference="left_wheel_rim_link">
-        <material>Gazebo/Red</material>
-    </gazebo>
     <!--  ########################### -->
     <!--  FRONT RIGHT WHEEL LINK -->
@@ -76,27 +73,16 @@
         <parent link="base_chassis_link"/>
         <child link="right_wheel_link"/>
-        <origin xyz="0 -0.17 0" rpy="${-pi/2} 0 0"/>
+        <origin xyz="0 -0.2 0" rpy="${-pi/2} 0 0"/>
         <axis xyz="0 0 1"/>
     </joint>
     <link name="right_wheel_link">
-        <xacro:insert_drive_wheel/>
+        <xacro:insert_mesh_drive_wheel/>
     </link>
     <xacro:gazebo_wheel_settings name="right_wheel_link"/>
-    <joint name="right_wheel_rim_joint" type="fixed">
-        <parent link="right_wheel_link"/>
-        <child link="right_wheel_rim_link"/>
-        <origin xyz="0 0 0" rpy="0 0 0"/>
-    </joint>
-    <link name="right_wheel_rim_link">
-        <xacro:insert_wheel_rim/>
-    </link>
-    <gazebo reference="right_wheel_rim_link">
-        <material>Gazebo/Red</material>
-    </gazebo>
     <!--  CASTER WHEEL LINK -->
     <joint name="caster_wheel_joint" type="fixed">
         <parent link="base_chassis_link"/>
         <child link="caster_wheel_link"/>
-        <origin xyz="-0.20 0 0"/>
+        <origin xyz="-0.18 0 0"/>
     </joint>
     <link name="caster_wheel_link">
@@ -114,5 +100,5 @@
             </geometry>
         </collision>
-        <xacro:inertial_sphere mass="0.2" radius="0.05">
+        <xacro:inertial_sphere mass="0.5" radius="0.05">
             <origin xyz="0 0 0" rpy="0 0 0"/>
         </xacro:inertial_sphere>
@@ -123,6 +109,6 @@
         <!-- <kp>1000000.0</kp>
         <kd>1.0</kd>
-        <fdir1>1 0 0</fdir1>
-        <minDepth>0.1</minDepth> -->
+        <fdir1>1 0 0</fdir1> -->
+        <minDepth>0.01</minDepth>
         <material>Gazebo/Grey</material>
     </gazebo>

File: mobo_bot_description/urdf/ros_controllers.xacro (robot description, xacro)
@@ -27,9 +27,9 @@
                 <right_joint>right_wheel_joint</right_joint>
                 <!-- kinematics -->
-                <wheel_separation>0.34</wheel_separation>
+                <wheel_separation>0.4</wheel_separation>
                 <wheel_diameter>0.1</wheel_diameter>
                 <!-- limits -->
                 <max_wheel_torque>100</max_wheel_torque>
-                <max_wheel_acceleration>5.0</max_wheel_acceleration>
+                <max_wheel_acceleration>4.0</max_wheel_acceleration>
                 <command_topic>cmd_vel</command_topic>
                 <!-- output -->

File: mobo_bot_description/urdf/sensors/cam.xacro (robot description, xacro)
@@ -3,5 +3,5 @@
     <!-- <xacro:arg name="cam_visual"   default="false"/> -->
     <xacro:property name="line_sense_angle"   value="${pi/2.5}"/>
-    <xacro:property name="line_sense_mode"   value="true"/>
+    <xacro:property name="line_sense_mode"   value="false"/>
     <!-- CAMERA LINK FRAME -->
     <joint name="cam_joint" type="fixed">
@@ -9,5 +9,5 @@
         <child link="cam_link"/>
         <xacro:if value="${line_sense_mode}">
-            <origin xyz="0.16 0 ${base_chassis_height+0.01}" rpy="0 ${line_sense_angle} 0"/>
+            <origin xyz="0.16 0 0" rpy="0 ${line_sense_angle} 0"/>
         </xacro:if>
         <xacro:unless value="${line_sense_mode}">

File: mobo_bot_description/urdf/sensors/sonar.xacro (robot description, xacro)
@@ -8,5 +8,5 @@
         <parent link="base_chassis_link"/>
         <child link="sonar_link"/>
-        <origin xyz="0.15 0 ${base_chassis_height/2}" rpy="0 0 0"/>
+        <origin xyz="0.16 0 ${base_chassis_height/2}" rpy="0 0 0"/>
         <axis xyz="0 0 0"/>
     </joint>
@@ -15,5 +15,5 @@
             <origin xyz="-0.005 0 0" rpy="0 ${pi/2} 0"/>
             <geometry>
-                <cylinder radius="0.01" length="0.01" />
+                <cylinder radius="0.015" length="0.01" />
             </geometry>
             <material name="blue"/>
@@ -22,5 +22,5 @@
             <origin xyz="-0.005 0 0" rpy="0 ${pi/2} 0"/>
             <geometry>
-                <cylinder radius="0.01" length="0.01" />
+                <cylinder radius="0.015" length="0.01" />
             </geometry>
         </collision>
