Commit message: cleaned up mobo_bot urdf file

File: mobo_bot_description/urdf/robot_urdf.xacro (robot description, xacro)
@@ -2,12 +2,198 @@
 <robot name="mobo_bot" xmlns:xacro="http://www.ros.org/wiki/xacro">
     <xacro:arg name="run_gz_sim" default="false"/>
-    <xacro:include filename="$(find mobo_bot_description)/urdf/color_macros.xacro" />
-    <xacro:include filename="$(find mobo_bot_description)/urdf/inertia_macros.xacro" />
-    <xacro:include filename="$(find mobo_bot_description)/urdf/robot_core.xacro" />
+    <material name="orange">
+        <color rgba="1 0.55 0 1"/>
+    </material>
+    <material name="black">
+        <color rgba="0.1 0.1 0.1 1"/>
+    </material>
+    <material name="silver">
+        <color rgba="0.6 0.6 0.6 1"/>
+    </material>
+    <material name="grey">
+        <color rgba="0.25 0.25 0.25 1"/>
+    </material>
+    <material name="blue">
+        <color rgba="0.2 0.2 1 1"/>
+    </material>
+    <material name="red">
+        <color rgba="1 0.1 0.1 1"/>
+    </material>
+    <xacro:macro name="inertial_sphere" params="mass radius *origin">
+        <inertial>
+            <xacro:insert_block name="origin"/>
+            <mass value="${mass}" />
+            <inertia ixx="${(2/5) * mass * (radius*radius)}" ixy="0.0" ixz="0.0"
+                    iyy="${(2/5) * mass * (radius*radius)}" iyz="0.0"
+                    izz="${(2/5) * mass * (radius*radius)}" />
+        </inertial>
+    </xacro:macro>
+    <xacro:macro name="inertial_box" params="mass x y z *origin">
+        <inertial>
+            <xacro:insert_block name="origin"/>
+            <mass value="${mass}" />
+            <inertia ixx="${(1/12) * mass * (y*y+z*z)}" ixy="0.0" ixz="0.0"
+                    iyy="${(1/12) * mass * (x*x+z*z)}" iyz="0.0"
+                    izz="${(1/12) * mass * (x*x+y*y)}" />
+        </inertial>
+    </xacro:macro>
+    <xacro:macro name="inertial_cylinder" params="mass length radius *origin">
+        <inertial>
+            <xacro:insert_block name="origin"/>
+            <mass value="${mass}" />
+            <inertia ixx="${(1/12) * mass * (3*radius*radius + length*length)}" ixy="0.0" ixz="0.0"
+                    iyy="${(1/12) * mass * (3*radius*radius + length*length)}" iyz="0.0"
+                    izz="${(1/2) * mass * (radius*radius)}" />
+        </inertial>
+    </xacro:macro>
+    <xacro:include filename="$(find mobo_bot_description)/urdf/urdf_models/box_with_fillet_macro.xacro"/>
+    <xacro:include filename="$(find mobo_bot_description)/urdf/urdf_models/drive_wheel_macro.xacro"/>
+    <xacro:include filename="$(find mobo_bot_description)/urdf/urdf_models/drive_wheel_rim_macro.xacro"/>
+    <xacro:include filename="$(find mobo_bot_description)/urdf/urdf_models/sonar.xacro"/>
+    <xacro:include filename="$(find mobo_bot_description)/urdf/urdf_models/lidar.xacro"/>
+    <xacro:include filename="$(find mobo_bot_description)/urdf/urdf_models/cam.xacro"/>
+    <xacro:property name="chassis_length" value="0.21"/>
+    <xacro:property name="chassis_width" value="0.21"/>
+    <xacro:property name="chassis_height" value="0.06"/>
+    <xacro:property name="slab_height" value="0.005"/>
+    <xacro:property name="chassis_mass" value="2.0"/>
+    <xacro:property name="chassis_color" value="orange"/>
+    <xacro:property name="wheel_seperation" value="0.24"/>
+    <xacro:property name="wheel_radius" value="0.034"/>
+    <xacro:property name="wheel_width" value="0.026"/>
+    <xacro:property name="wheel_mass" value="0.08"/>
+    <xacro:property name="wheel_height_offset" value="0.024"/>
+    <xacro:property name="castor_wheel_diameter" value="${wheel_radius+wheel_height_offset}"/>
+    <xacro:property name="castor_wheel_mass" value="0.08"/>
+    <link name="base_link">
+    </link>
+    <joint name="chassis_joint" type="fixed">
+        <parent link="base_link"/>
+        <child link="chassis"/>
+        <origin xyz="0 0 ${wheel_radius+wheel_height_offset}"/>
+    </joint>
+    <link name="chassis">
+        <xacro:insert_box_with_fillet x="-0.040" y="0" z="0"
+            size_x="${chassis_length}" size_y="${chassis_width}" size_z="${slab_height}"
+            fillet_radius="0.04"/>
+        <xacro:insert_box_with_fillet x="-0.040" y="0" z="${chassis_height}"
+            size_x="${chassis_length}" size_y="${chassis_width}" size_z="${slab_height}"
+            fillet_radius="0.04"/>
+        <visual>
+            <origin xyz="0.04 0.08 ${chassis_height/2}" rpy="0 0 0"/>
+            <geometry>
+                <cylinder radius="0.005" length="${chassis_height}"/>
+            </geometry>
+            <material name="orange"/>
+        </visual>
+        <visual>
+            <origin xyz="0.04 -0.08 ${chassis_height/2}" rpy="0 0 0"/>
+            <geometry>
+                <cylinder radius="0.005" length="${chassis_height}"/>
+            </geometry>
+            <material name="orange"/>
+        </visual>
+        <visual>
+            <origin xyz="-0.11 0.08 ${chassis_height/2}" rpy="0 0 0"/>
+            <geometry>
+                <cylinder radius="0.005" length="${chassis_height}"/>
+            </geometry>
+            <material name="orange"/>
+        </visual>
+        <visual>
+            <origin xyz="-0.11 -0.08 ${chassis_height/2}" rpy="0 0 0"/>
+            <geometry>
+                <cylinder radius="0.005" length="${chassis_height}"/>
+            </geometry>
+            <material name="orange"/>
+        </visual>
+        <collision>
+           <origin xyz="-0.02 0 ${chassis_height/2}" rpy="0 0 0"/>
+            <geometry>
+                <box size="${chassis_length} ${chassis_width} ${chassis_height}"/>
+            </geometry>
+        </collision>
+        <xacro:inertial_box mass="${chassis_mass}" x="${chassis_length}" y="${chassis_width}" z="${chassis_height}">
+            <origin xyz="-0.06 0 ${chassis_height/2}" rpy="0 0 0"/>
+        </xacro:inertial_box>
+    </link>
+    <xacro:insert_drive_wheel
+        base_name="left_wheel"
+        parent_name="base_link"
+        x="0" y="${wheel_seperation/2}" z="${wheel_radius}"
+        mass="${wheel_mass}"
+        radius="${wheel_radius}"
+        thickness="${wheel_width}"/>
+    <xacro:insert_drive_wheel_rim
+        base_name="left_rim"
+        parent_name="left_wheel"
+        radius="${wheel_radius}"
+        thickness="${wheel_width}"
+        spoke_width="0.005"/>
+    <xacro:insert_drive_wheel
+        base_name="right_wheel"
+        parent_name="base_link"
+        x="0" y="${-wheel_seperation/2}" z="${wheel_radius}"
+        mass="${wheel_mass}"
+        radius="${wheel_radius}"
+        thickness="${wheel_width}"/>
+    <xacro:insert_drive_wheel_rim
+        base_name="right_rim"
+        parent_name="right_wheel"
+        radius="${wheel_radius}"
+        thickness="${wheel_width}"
+        spoke_width="0.005"/>
+    <joint name="castor_wheel_joint" type="fixed">
+        <parent link="base_link"/>
+        <child link="castor_wheel"/>
+        <origin xyz="-0.1 0 ${castor_wheel_diameter/2}"/>
+    </joint>
+    <link name="castor_wheel">
+        <visual>
+            <origin xyz="0 0 0" rpy="0 0 0"/>
+            <geometry>
+                <sphere radius="${castor_wheel_diameter/2}" />
+            </geometry>
+            <material name="grey">
+                <color rgba="0.25 0.25 0.25 1"/>
+            </material>
+        </visual>
+        <collision>
+           <origin xyz="0 0 0" rpy="0 0 0"/>
+            <geometry>
+                <sphere radius="${castor_wheel_diameter/2}" />
+            </geometry>
+        </collision>
+        <xacro:inertial_sphere mass="${castor_wheel_mass}" radius="${castor_wheel_diameter/2}">
+            <origin xyz="0 0 0" rpy="0 0 0"/>
+        </xacro:inertial_sphere>
+    </link>
+    <xacro:property name="lidar_z_offset" value="0.04"/>
+    <xacro:insert_lidar
+        base_name="lidar"
+        parent_name="chassis"
+        x="0.01" y="0" z="${chassis_height+lidar_z_offset}"
+        mass="0.1"/>
+    <joint name="imu_joint" type="fixed">
+        <parent link="chassis"/>
+        <child link="imu"/>
+        <origin xyz="0 0 ${chassis_height}"/>
+    </joint>
+    <link name="imu"></link>
+    <xacro:insert_sonar
+        base_name="sonar"
+        parent_name="chassis"
+        x="0.065" y="0" z="${chassis_height/6}"
+        mass="0.005"/>
+    <xacro:insert_camera
+        base_name="camera"
+        parent_name="chassis"
+        x="0.075" y="0" z="${chassis_height+0.015}"
+        mass="0.005" tilt_angle="0.00"/>
     <xacro:if value="$(arg run_gz_sim)">
-        <xacro:include filename="$(find mobo_bot_description)/urdf/controllers/gazebo_diff_drive_control.xacro" />
+        <xacro:include filename="$(find mobo_bot_description)/urdf/gazebo_properties.xacro" />
     </xacro:if>
     <xacro:unless value="$(arg run_gz_sim)">
-        <xacro:include filename="$(find mobo_bot_description)/urdf/controllers/epmc_diff_drive_ros2_control.xacro" />
+        <xacro:include filename="$(find mobo_bot_description)/urdf/epmc_ros2_control.xacro" />
     </xacro:unless>
 </robot>

File: mobo_bot_description/urdf/urdf_models/cam.xacro (robot description, xacro)
@@ -9,16 +9,7 @@
         <link name="${base_name}">
             <visual>
-                <origin xyz="-0.005 0 0" rpy="0 ${-pi/2} 0"/>
+                <origin xyz="-0.01 0 0" rpy="0 0 0"/>
                 <geometry>
-                    <cylinder radius="0.007" length="0.01"/>
-                </geometry>
-                <material name="grey">
-                    <color rgba="0.25 0.25 0.25 1"/>
-                </material>
-            </visual>
-            <visual>
-                <origin xyz="-0.01 0 0" rpy="0 ${-pi/2} 0"/>
-                <geometry>
-                    <box size="0.02 0.03 0.01"/>
+                    <box size="0.02 0.06 0.02"/>
                 </geometry>
                 <material name="grey">
@@ -27,12 +18,12 @@
             </visual>
             <collision>
-                <origin xyz="-0.005 0 0" rpy="0 ${-pi/2} 0"/>
+                <origin xyz="-0.01 0 0" rpy="0 0 0"/>
                 <geometry>
-                    <cylinder radius="0.01" length="0.01"/>
+                    <box size="0.02 0.06 0.02"/>
                 </geometry>
             </collision>
-            <xacro:inertial_cylinder mass="${mass}" radius="0.01" length="0.01">
-                <origin xyz="-0.005 0 0" rpy="0 ${-pi/2} 0"/>
-            </xacro:inertial_cylinder>
+            <xacro:inertial_box mass="${mass}" x="0.02" y="0.06" z="0.02">
+                <origin xyz="-0.01 0 0" rpy="0 0 0"/>
+            </xacro:inertial_box>
         </link>
         <joint name="${base_name}_optical_joint" type="fixed">
