Commit message: update robot description

File: mobo_bot_description/urdf/other_parts/box_with_fillet_macro.xacro (robot description, xacro)
@@ -1,5 +1,5 @@
 <?xml version="1.0"?>
 <robot xmlns:xacro="http://www.ros.org/wiki/xacro" >
-    <xacro:macro name="insert_box_with_fillet" params="x y z size_x size_y size_z fillet_radius material">
+    <xacro:macro name="insert_box_with_fillet" params="x y z size_x size_y size_z fillet_radius color">
             <!-- logitudinal box -->
             <visual>
@@ -8,5 +8,5 @@
                     <box size="${size_x} ${size_y-(2*fillet_radius)} ${size_z}"/>
                 </geometry>
-                <material name="${material}"/>
+                <material name="${color}"/>
             </visual>
             <!-- lateral box -->
@@ -16,5 +16,5 @@
                     <box size="${size_x-(2*fillet_radius)} ${size_y} ${size_z}"/>
                 </geometry>
-                <material name="${material}"/>
+                <material name="${color}"/>
             </visual>
             <!-- cylinder1 -->
@@ -24,5 +24,5 @@
                     <cylinder length="${size_z}" radius="${fillet_radius}"/>
                 </geometry>
-                <material name="${material}"/>
+                <material name="${color}"/>
             </visual>
             <!-- cylinder2 -->
@@ -32,5 +32,5 @@
                     <cylinder length="${size_z}" radius="${fillet_radius}"/>
                 </geometry>
-                <material name="${material}"/>
+                <material name="${color}"/>
             </visual>
             <!-- cylinder3 -->
@@ -40,5 +40,5 @@
                     <cylinder length="${size_z}" radius="${fillet_radius}"/>
                 </geometry>
-                <material name="${material}"/>
+                <material name="${color}"/>
             </visual>
             <!-- cylinder4 -->
@@ -48,5 +48,5 @@
                     <cylinder length="${size_z}" radius="${fillet_radius}"/>
                 </geometry>
-                <material name="${material}"/>
+                <material name="${color}"/>
             </visual>
     </xacro:macro>

File: mobo_bot_description/urdf/other_parts/drive_wheel_macro.xacro (robot description, xacro)
@@ -15,18 +15,5 @@
         </inertial>
     </xacro:macro>
-     <!-- GAZEBO WHEEL PARAMETERS -->
-    <xacro:macro name="gazebo_wheel_settings" params="name">
-        <gazebo reference="${name}">
-            <mu1>1.0</mu1>
-            <mu2>1.0</mu2>
-            <!-- <kp>1000000</kp> -->
-            <!-- <kd>0.001</kd> -->
-            <minDepth>0.005</minDepth>
-            <!-- <fdir1>${fdir}</fdir1> -->
-            <material>Gazebo/FlatBlack</material>
-        </gazebo>
-    </xacro:macro>
-    <!--  ########################### -->
-    <xacro:macro name="insert_drive_wheel" params="base_name parent_name x y z mass radius thickness">
+    <xacro:macro name="insert_drive_wheel" params="base_name parent_name x y z mass radius thickness color">
         <joint name="${base_name}_joint" type="continuous">
             <parent link="${parent_name}"/>
@@ -41,5 +28,5 @@
                     <cylinder radius="${radius}" length="${thickness}"/>
                 </geometry>
-                <xacro:material_black/>
+                <material name="${color}"/>
             </visual>
             <collision>
@@ -54,5 +41,4 @@
             </xacro:inertial_cylinder>
         </link>
-        <xacro:gazebo_wheel_settings name="${base_name}"/>
     </xacro:macro>
 </robot>

File: mobo_bot_description/urdf/other_parts/drive_wheel_rim_macro.xacro (robot description, xacro)
@@ -1,14 +1,9 @@
 <?xml version="1.0"?>
 <robot xmlns:xacro="http://www.ros.org/wiki/xacro" >
-    <xacro:macro name="material_red">
-        <material name="red">
-            <color rgba="1 0 0 1"/>
-        </material>
-    </xacro:macro>
-    <xacro:macro name="insert_drive_wheel_rim" params="base_name parent_name x y z radius thickness spoke_width">
+    <xacro:macro name="insert_drive_wheel_rim" params="base_name parent_name radius thickness spoke_width color">
         <joint name="${base_name}_joint" type="fixed">
             <parent link="${parent_name}"/>
             <child link="${base_name}"/>
-            <origin xyz="${x} ${y} ${z}" rpy="0 0 0"/>
+            <origin xyz="0 0 0" rpy="0 0 0"/>
         </joint>
         <link name="${base_name}">
@@ -16,33 +11,30 @@
                 <origin xyz="0 0 0" rpy="0 0 0"/>
                 <geometry>
-                    <box size="${spoke_width} ${radius*1.2} ${thickness}"/>
+                    <box size="${spoke_width} ${radius*1.3} ${thickness+0.001}"/>
                 </geometry>
-                <xacro:material_red/>
+                <material name="${color}"/>
             </visual>
             <visual>
                 <origin xyz="0 0 0" rpy="0 0 ${pi/2}"/>
                 <geometry>
-                    <box size="${spoke_width} ${radius*1.2} ${thickness}"/>
+                    <box size="${spoke_width} ${radius*1.3} ${thickness+0.001}"/>
                 </geometry>
-                <xacro:material_red/>
+                <material name="${color}"/>
             </visual>
             <visual>
                 <origin xyz="0 0 0" rpy="0 0 ${-pi/4}"/>
                 <geometry>
-                    <box size="${spoke_width} ${radius*1.2} ${thickness}"/>
+                    <box size="${spoke_width} ${radius*1.3} ${thickness+0.001}"/>
                 </geometry>
-                <xacro:material_red/>
+                <material name="${color}"/>
             </visual>
             <visual>
                 <origin xyz="0 0 0" rpy="0 0 ${pi/4}"/>
                 <geometry>
-                    <box size="${spoke_width} ${radius*1.2} ${thickness}"/>
+                    <box size="${spoke_width} ${radius*1.3} ${thickness+0.001}"/>
                 </geometry>
-                <xacro:material_red/>
+                <material name="${color}"/>
             </visual>
         </link>
-        <gazebo reference="${base_name}">
-            <material>Gazebo/Red</material>
-        </gazebo>
     </xacro:macro>
 </robot>

File: mobo_bot_description/urdf/robot_core.xacro (robot description, xacro)
@@ -8,9 +8,9 @@
     <!-- <xacro:include filename="$(find mobo_bot_description)/urdf/sensors/imu.xacro"/> -->
     <!-- <xacro:include filename="$(find mobo_bot_description)/urdf/sensors/cam.xacro"/> -->
-    <xacro:property name="chassis_length" value="0.24"/>
-    <xacro:property name="chassis_width" value="0.23"/>
+    <xacro:property name="chassis_length" value="0.21"/>
+    <xacro:property name="chassis_width" value="0.21"/>
     <xacro:property name="chassis_height" value="0.06"/>
-    <xacro:property name="chassis_mass" value="3.0"/>
-    <xacro:property name="wheel_seperation" value="0.25"/>
+    <xacro:property name="chassis_mass" value="2.0"/>
+    <xacro:property name="wheel_seperation" value="0.23"/>
     <xacro:property name="wheel_radius" value="0.034"/>
     <xacro:property name="wheel_width" value="0.014"/>
@@ -30,7 +30,7 @@
     </joint>
     <link name="chassis">
-        <xacro:insert_box_with_fillet x="-0.02" y="0" z="${chassis_height/2}"
+        <xacro:insert_box_with_fillet x="-0.025" y="0" z="${chassis_height/2}"
             size_x="${chassis_length}" size_y="${chassis_width}" size_z="${chassis_height}"
-            fillet_radius="0.05" material="white"/>
+            fillet_radius="0.05" color="orange"/>
         <collision>
            <origin xyz="-0.02 0 ${chassis_height/2}" rpy="0 0 0"/>
@@ -43,7 +43,9 @@
         </xacro:inertial_box>
     </link>
-    <gazebo reference="chassis">
-        <material>Gazebo/White</material>
-    </gazebo>
+    <xacro:if value="$(arg use_simulation)">
+        <gazebo reference="chassis">
+            <material>Gazebo/Orange</material>
+        </gazebo>
+    </xacro:if>
     <!--  ########################### -->
     <!-- LEFT DRIVE WHEEL -->
@@ -54,12 +56,29 @@
         mass="${wheel_mass}"
         radius="${wheel_radius}"
-        thickness="${wheel_width}"/>
+        thickness="${wheel_width}"
+        color="black"/>
+    <xacro:if value="$(arg use_simulation)">
+        <gazebo reference="left_wheel">
+            <mu1>1.0</mu1>
+            <mu2>1.0</mu2>
+            <!-- <kp>1000000</kp> -->
+            <!-- <kd>0.001</kd> -->
+            <minDepth>0.005</minDepth>
+            <!-- <fdir1>${fdir}</fdir1> -->
+            <material>Gazebo/FlatBlack</material>
+        </gazebo>
+    </xacro:if>
     <xacro:insert_drive_wheel_rim
         base_name="left_rim"
         parent_name="left_wheel"
-        x="0" y="0" z="0.001"
         radius="${wheel_radius}"
         thickness="${wheel_width}"
-        spoke_width="0.005"/>
+        spoke_width="0.005"
+        color="red"/>
+    <xacro:if value="$(arg use_simulation)">
+        <gazebo reference="left_rim">
+            <material>Gazebo/Red</material>
+        </gazebo>
+    </xacro:if>
     <!-- ############################# -->
     <!-- RIGHT DRIVE WHEEL -->
@@ -70,12 +89,29 @@
         mass="${wheel_mass}"
         radius="${wheel_radius}"
-        thickness="${wheel_width}"/>
+        thickness="${wheel_width}"
+        color="black"/>
+    <xacro:if value="$(arg use_simulation)">
+        <gazebo reference="right_wheel">
+            <mu1>1.0</mu1>
+            <mu2>1.0</mu2>
+            <!-- <kp>1000000</kp> -->
+            <!-- <kd>0.001</kd> -->
+            <minDepth>0.005</minDepth>
+            <!-- <fdir1>${fdir}</fdir1> -->
+            <material>Gazebo/FlatBlack</material>
+        </gazebo>
+    </xacro:if>
     <xacro:insert_drive_wheel_rim
         base_name="right_rim"
         parent_name="right_wheel"
-        x="0" y="0" z="-0.001"
         radius="${wheel_radius}"
         thickness="${wheel_width}"
-        spoke_width="0.005"/>
+        spoke_width="0.005"
+        color="red"/>
+    <xacro:if value="$(arg use_simulation)">
+        <gazebo reference="right_rim">
+            <material>Gazebo/Red</material>
+        </gazebo>
+    </xacro:if>
     <!-- ############################# -->
     <!--  castor WHEEL LINK -->
@@ -83,5 +119,5 @@
         <parent link="base_link"/>
         <child link="castor_wheel"/>
-        <origin xyz="-0.1 0 ${castor_wheel_radius}"/>
+        <origin xyz="-0.095 0 ${castor_wheel_radius}"/>
     </joint>
     <link name="castor_wheel">
@@ -103,13 +139,15 @@
         </xacro:inertial_sphere>
     </link>
-    <gazebo reference="castor_wheel">
-        <mu1>0.001</mu1>
-        <mu2>0.001</mu2>
-        <!-- <kp>1000000.0</kp> -->
-        <!-- <kd>1.0</kd> -->
-        <!-- <fdir1>1 0 0</fdir1> -->
-        <!-- <minDepth>0.01</minDepth> -->
-        <material>Gazebo/Grey</material>
-    </gazebo>
+    <xacro:if value="$(arg use_simulation)">
+        <gazebo reference="castor_wheel">
+            <mu1>0.001</mu1>
+            <mu2>0.001</mu2>
+            <!-- <kp>1000000.0</kp> -->
+            <!-- <kd>1.0</kd> -->
+            <!-- <fdir1>1 0 0</fdir1> -->
+            <!-- <minDepth>0.01</minDepth> -->
+            <material>Gazebo/Grey</material>
+        </gazebo>
+    </xacro:if>
     <!--  ########################### -->
     <!--  sonar -->
@@ -117,8 +155,47 @@
         base_name="sonar"
         parent_name="chassis"
-        x="0.1" y="0" z="${chassis_height/2}"
-        mass="0.005"
-        min_range="0.02" max_range="3.0"
-        resolution="0.01" visualize="false"/>
+        x="0.0825" y="0" z="${chassis_height/2}"
+        mass="0.005" color="blue"/>
+    <xacro:if value="$(arg use_simulation)">
+        <gazebo reference="sonar">
+            <material>Gazebo/Blue</material>
+            <sensor name="sonar" type="ray">
+                <always_on>true</always_on>
+                <visualize>false</visualize>
+                <pose>0.0 0 0.0 0 0 0</pose>
+                <update_rate>10</update_rate>
+                <ray>
+                    <scan>
+                        <horizontal>
+                            <samples>20</samples>
+                            <resolution>1</resolution>
+                            <min_angle>${-pi/90}</min_angle>
+                            <max_angle>${pi/90}</max_angle>
+                        </horizontal>
+                        <vertical>
+                            <samples>20</samples>
+                            <resolution>1</resolution>
+                            <min_angle>${-pi/150}</min_angle>
+                            <max_angle>${pi/150}</max_angle>
+                        </vertical>
+                    </scan>
+                    <range>
+                        <min>0.01</min>
+                        <max>0.4</max>
+                        <resolution>0.01</resolution>
+                    </range>
+                </ray>
+                <plugin name="sonar_plugin" filename="libgazebo_ros_ray_sensor.so">
+                    <ros>
+                        <namespace>sonar</namespace>
+                        <remapping>~/out:=range</remapping>
+                    </ros>
+                    <output_type>sensor_msgs/Range</output_type>
+                    <radiation_type>ultrasound</radiation_type>
+                    <frame_name>sonar</frame_name>
+                </plugin>
+            </sensor>
+        </gazebo>
+    </xacro:if>
      <!--  lidar -->
     <xacro:property name="lidar_z_offset" value="0.04"/>
@@ -126,25 +203,136 @@
         base_name="lidar"
         parent_name="chassis"
-        x="0.02" y="0" z="${chassis_height+lidar_z_offset}"
-        mass="0.1" samples="360"
-        min_angle="${-pi*2}" max_angle="${pi*2}"
-        min_range="0.1" max_range="10"
-        visualize="false"/>
+        x="0.01" y="0" z="${chassis_height+lidar_z_offset}"
+        mass="0.1" color="grey"/>
+    <xacro:if value="$(arg use_simulation)">
+        <gazebo reference="right_rim">
+            <material>Gazebo/Red</material>
+        </gazebo>
+    </xacro:if>
+    <gazebo reference="lidar">
+        <material>Gazebo/DarkGrey</material>
+        <sensor name="lidar" type="ray">
+            <pose> 0 0 0 0 0 0 </pose>
+            <visualize>false</visualize>
+            <update_rate>10</update_rate>
+            <ray>
+                <scan>
+                    <horizontal>
+                        <samples>360</samples>
+                        <min_angle>${-pi*2}</min_angle>
+                        <max_angle>${pi*2}</max_angle>
+                    </horizontal>
+                </scan>
+                <range>
+                    <min>0.1</min>
+                    <max>10.0</max>
+                </range>
+            </ray>
+            <plugin name="lidar_plugin" filename="libgazebo_ros_ray_sensor.so">
+                <ros>
+                    <namespace>lidar</namespace>
+                    <remapping>~/out:=scan</remapping>
+                </ros>
+                <output_type>sensor_msgs/LaserScan</output_type>
+                <frame_name>lidar</frame_name>
+            </plugin>
+        </sensor>
+    </gazebo>
     <!--  imu -->
     <!-- <xacro:insert_imu
         base_name="imu"
         parent_name="chassis"
-        x="0" y="0" z="${chassis_height}"/> -->
+        x="0" y="0" z="${chassis_height}"/>
+    <xacro:if value="$(arg use_simulation)">
+        <gazebo reference="imu">
+            <sensor name="imu" type="imu">
+                <always_on>true</always_on>
+                <update_rate>30</update_rate>
+                <visualize>true</visualize>
+                <imu>
+                    <angular_velocity>
+                        <x>
+                            <noise type="gaussian">
+                                <mean>0.0</mean>
+                                <stddev>2e-4</stddev>
+                            </noise>
+                        </x>
+                        <y>
+                            <noise type="gaussian">
+                                <mean>0.0</mean>
+                                <stddev>2e-4</stddev>
+                            </noise>
+                        </y>
+                        <z>
+                            <noise type="gaussian">
+                                <mean>0.0</mean>
+                                <stddev>2e-4</stddev>
+                            </noise>
+                        </z>
+                    </angular_velocity>
+                    <linear_acceleration>
+                        <x>
+                            <noise type="gaussian">
+                                <mean>0.0</mean>
+                                <stddev>1.7e-2</stddev>
+                            </noise>
+                        </x>
+                        <y>
+                            <noise type="gaussian">
+                                <mean>0.0</mean>
+                                <stddev>1.7e-2</stddev>
+                            </noise>
+                        </y>
+                        <z>
+                            <noise type="gaussian">
+                                <mean>0.0</mean>
+                                <stddev>1.7e-2</stddev>
+                            </noise>
+                        </z>
+                    </linear_acceleration>
+                </imu>
+                <plugin name="imu_plugin" filename="libgazebo_ros_imu_sensor.so">
+                    <ros>
+                        <namespace>imu</namespace>
+                        <remapping>~/out:=data</remapping>
+                    </ros>
+                    <initial_orientation_as_reference>false</initial_orientation_as_reference>
+                    <frame_name>imu</frame_name>
+                </plugin>
+            </sensor>
+        </gazebo>
+    </xacro:if> -->
     <!-- camera -->
-    <!-- <xacro:property name="cam_x_offset" value="0.04"/>
-    <xacro:property name="cam_z_offset" value="0.02"/>
+    <!-- <xacro:property name="cam_x_offset" value="0.015"/>
+    <xacro:property name="cam_z_offset" value="0.01"/>
     <xacro:insert_camera
         base_name="camera"
         parent_name="chassis"
-        x="${(chassis_length*0.375)+cam_x_offset}" y="0" z="${chassis_height+cam_z_offset}"
-        mass="0.005"
-        width="320" height="240"
-        min_range="0.02" max_range="5.0"
-        tilt_angle="0"
-        visualize="true"/> -->
+        x="${0.08+cam_x_offset}" y="0" z="${chassis_height+cam_z_offset}"
+        mass="0.005" tilt_angle="0" color="grey"/>
+    <xacro:if value="$(arg use_simulation)">
+        <gazebo reference="camera">
+          <material>Gazebo/DarkGrey</material>
+          <sensor name="camera" type="camera">
+            <pose> 0 0 0 0 0 0 </pose>
+            <visualize>false</visualize>
+            <update_rate>20</update_rate>
+            <camera>
+                <horizontal_fov>1.46608</horizontal_fov>
+                <image>
+                    <format>R8G8B8</format>
+                    <width>320</width>
+                    <height>240</height>
+                </image>
+                <clip>
+                    <near>0.02</near>
+                    <far>5.0</far>
+                </clip>
+            </camera>
+            <plugin name="camera_plugin" filename="libgazebo_ros_camera.so">
+                <frame_name>camera_optical_link</frame_name>
+            </plugin>
+          </sensor>
+        </gazebo>
+    </xacro:if> -->
 </robot>

File: mobo_bot_description/urdf/robot_urdf.xacro (robot description, xacro)
@@ -1,7 +1,19 @@
 <?xml version="1.0"?>
 <robot name="mobo_bot" xmlns:xacro="http://www.ros.org/wiki/xacro">
+    <!-- ########### ARGUMENTS ######################### -->
+    <xacro:arg name="use_simulation" default="false"/>
+    <!-- <xacro:arg name="laser_visual" default="false"/> -->
+    <!-- <xacro:arg name="imu_visual"   default="true"/> -->
+    <!-- <xacro:arg name="sonar_visual"   default="false"/> -->
+    <!-- <xacro:arg name="cam_visual"   default="false"/> -->
+    <!-- ############################################### -->
     <xacro:include filename="$(find mobo_bot_description)/urdf/color_macros.xacro" />
     <xacro:include filename="$(find mobo_bot_description)/urdf/inertia_macros.xacro" />
     <xacro:include filename="$(find mobo_bot_description)/urdf/robot_core.xacro" />
-    <xacro:include filename="$(find mobo_bot_description)/urdf/controllers/gazebo_control.xacro" />
+    <xacro:if value="$(arg use_simulation)">
+        <xacro:include filename="$(find mobo_bot_description)/urdf/controllers/gazebo_control.xacro" />
+    </xacro:if>
+    <xacro:unless value="$(arg use_simulation)">
+        <xacro:include filename="$(find mobo_bot_description)/urdf/controllers/epmc_ros2_control.xacro" />
+    </xacro:unless>
 </robot>
