Commit message: update robot description

File: mobo_bot_description/urdf/sensors/cam.xacro (robot description, xacro)
@@ -1,5 +1,5 @@
 <?xml version="1.0"?>
 <robot xmlns:xacro="http://www.ros.org/wiki/xacro" >
-    <xacro:macro name="insert_camera" params="base_name parent_name x y z mass width height min_range max_range tilt_angle visualize">
+    <xacro:macro name="insert_camera" params="base_name parent_name x y z mass tilt_angle color">
         <joint name="${base_name}_joint" type="fixed">
             <parent link="${parent_name}"/>
@@ -9,26 +9,25 @@
         <link name="${base_name}">
             <visual>
-                <origin xyz="-0.02 0 0" rpy="0 ${-pi/2} 0"/>
+                <origin xyz="-0.005 0 0" rpy="0 ${-pi/2} 0"/>
                 <geometry>
-                    <cylinder radius="0.015" length="0.04"/>
+                    <cylinder radius="0.007" length="0.01"/>
                 </geometry>
-                <material name="grey"/>
+                <material name="${color}"/>
             </visual>
             <visual>
-                <origin xyz="-0.03 0 0" rpy="0 ${-pi/2} 0"/>
+                <origin xyz="-0.01 0 0" rpy="0 ${-pi/2} 0"/>
                 <geometry>
-                    <!-- <cylinder radius="0.03" length="0.02"/> -->
-                    <box size="0.04 0.06 0.02"/>
+                    <box size="0.02 0.03 0.01"/>
                 </geometry>
-                <material name="grey"/>
+                <material name="${color}"/>
             </visual>
             <collision>
-                <origin xyz="-0.02 0 0" rpy="0 ${-pi/2} 0"/>
+                <origin xyz="-0.005 0 0" rpy="0 ${-pi/2} 0"/>
                 <geometry>
-                    <cylinder radius="0.02" length="0.04"/>
+                    <cylinder radius="0.01" length="0.01"/>
                 </geometry>
             </collision>
-            <xacro:inertial_cylinder mass="${mass}" radius="0.02" length="0.04">
-                <origin xyz="-0.02 0 0" rpy="0 ${-pi/2} 0"/>
+            <xacro:inertial_cylinder mass="${mass}" radius="0.01" length="0.01">
+                <origin xyz="-0.005 0 0" rpy="0 ${-pi/2} 0"/>
             </xacro:inertial_cylinder>
         </link>
@@ -39,28 +38,4 @@
         </joint>
         <link name="${base_name}_optical_link"/>
-        <gazebo reference="${base_name}">
-          <material>Gazebo/DarkGrey</material>
-          <sensor name="${base_name}" type="camera">
-            <pose> 0 0 0 0 0 0 </pose>
-            <visualize>${visualize}</visualize>
-            <update_rate>20</update_rate>
-            <camera>
-                <!-- <horizontal_fov>1.089</horizontal_fov> -->
-                <horizontal_fov>1.46608</horizontal_fov>
-                <image>
-                    <format>R8G8B8</format>
-                    <width>${width}</width>
-                    <height>${height}</height>
-                </image>
-                <clip>
-                    <near>${min_range}</near>
-                    <far>${max_range}</far>
-                </clip>
-            </camera>
-            <plugin name="${base_name}_plugin" filename="libgazebo_ros_camera.so">
-                <frame_name>${base_name}_optical_link</frame_name>
-            </plugin>
-          </sensor>
-        </gazebo>
     </xacro:macro>
 </robot>

File: mobo_bot_description/urdf/sensors/imu.xacro (robot description, xacro)
@@ -8,61 +8,4 @@
         </joint>
         <link name="${base_name}"/>
-        <gazebo reference="${base_name}">
-            <sensor name="${base_name}" type="imu">
-                <always_on>true</always_on>
-                <update_rate>30</update_rate>
-                <visualize>true</visualize>
-                <imu>
-                    <angular_velocity>
-                        <x>
-                            <noise type="gaussian">
-                                <mean>0.0</mean>
-                                <stddev>2e-4</stddev>
-                            </noise>
-                        </x>
-                        <y>
-                            <noise type="gaussian">
-                                <mean>0.0</mean>
-                                <stddev>2e-4</stddev>
-                            </noise>
-                        </y>
-                        <z>
-                            <noise type="gaussian">
-                                <mean>0.0</mean>
-                                <stddev>2e-4</stddev>
-                            </noise>
-                        </z>
-                    </angular_velocity>
-                    <linear_acceleration>
-                        <x>
-                            <noise type="gaussian">
-                                <mean>0.0</mean>
-                                <stddev>1.7e-2</stddev>
-                            </noise>
-                        </x>
-                        <y>
-                            <noise type="gaussian">
-                                <mean>0.0</mean>
-                                <stddev>1.7e-2</stddev>
-                            </noise>
-                        </y>
-                        <z>
-                            <noise type="gaussian">
-                                <mean>0.0</mean>
-                                <stddev>1.7e-2</stddev>
-                            </noise>
-                        </z>
-                    </linear_acceleration>
-                </imu>
-                <plugin name="${base_name}_plugin" filename="libgazebo_ros_imu_sensor.so">
-                    <ros>
-                        <namespace>${base_name}</namespace>
-                        <remapping>~/out:=data</remapping>
-                    </ros>
-                    <initial_orientation_as_reference>false</initial_orientation_as_reference>
-                    <frame_name>${base_name}</frame_name>
-                </plugin>
-            </sensor>
-        </gazebo>
     </xacro:macro>
 </robot>

File: mobo_bot_description/urdf/sensors/lidar.xacro (robot description, xacro)
@@ -1,5 +1,5 @@
 <?xml version="1.0"?>
 <robot xmlns:xacro="http://www.ros.org/wiki/xacro" >
-    <xacro:macro name="insert_lidar" params="base_name parent_name x y z mass samples min_angle max_angle min_range max_range visualize">
+    <xacro:macro name="insert_lidar" params="base_name parent_name x y z mass color">
         <joint name="${base_name}_joint" type="fixed">
             <parent link="${parent_name}"/>
@@ -13,5 +13,5 @@
                     <cylinder radius="0.03" length="0.04"/>
                 </geometry>
-                <material name="grey"/>
+                <material name="${color}"/>
             </visual>
             <collision>
@@ -25,34 +25,4 @@
             </xacro:inertial_cylinder>
         </link>
-        <gazebo reference="${base_name}">
-            <material>Gazebo/DarkGrey</material>
-            <sensor name="${base_name}" type="ray">
-                <pose> 0 0 0 0 0 0 </pose>
-                <visualize>${visualize}</visualize>
-                <update_rate>10</update_rate>
-                <ray>
-                    <scan>
-                        <horizontal>
-                            <samples>${samples}</samples>
-                            <min_angle>${min_angle}</min_angle>
-                            <max_angle>${max_angle}</max_angle>
-                        </horizontal>
-                    </scan>
-                    <range>
-                        <min>${min_range}</min>
-                        <max>${max_range}</max>
-                    </range>
-                </ray>
-                <plugin name="${base_name}_plugin" filename="libgazebo_ros_ray_sensor.so">
-                    <ros>
-                        <namespace>${base_name}</namespace>
-                        <remapping>~/out:=scan</remapping>
-                        <!-- <argument>~/out:=scan</argument> -->
-                    </ros>
-                    <output_type>sensor_msgs/LaserScan</output_type>
-                    <frame_name>${base_name}</frame_name>
-                </plugin>
-            </sensor>
-        </gazebo>
     </xacro:macro>
 </robot>

File: mobo_bot_description/urdf/sensors/sonar.xacro (robot description, xacro)
@@ -4,5 +4,5 @@
     <!-- <xacro:property name="deg2rad" value="0.017460317"/>
     <xacro:property name="scan_angle" value="1"/> -->
-    <xacro:macro name="insert_sonar" params="base_name parent_name x y z mass min_range max_range resolution visualize">
+    <xacro:macro name="insert_sonar" params="base_name parent_name x y z mass color">
         <joint name="${base_name}_joint" type="fixed">
             <parent link="${parent_name}"/>
@@ -16,5 +16,5 @@
                     <cylinder radius="0.006" length="0.006"/>
                 </geometry>
-                <material name="blue"/>
+                <material name="${color}"/>
             </visual>
             <collision>
@@ -29,5 +29,5 @@
                     <cylinder radius="0.006" length="0.006"/>
                 </geometry>
-                <material name="blue"/>
+                <material name="${color}"/>
             </visual>
             <collision>
@@ -41,43 +41,4 @@
             </xacro:inertial_cylinder>
         </link>
-        <gazebo reference="${base_name}">
-            <material>Gazebo/Blue</material>
-            <sensor name="${base_name}" type="ray">
-                <always_on>true</always_on>
-                <visualize>${visualize}</visualize>
-                <pose>0.0 0 0.0 0 0 0</pose>
-                <update_rate>5</update_rate>
-                <ray>
-                    <scan>
-                        <horizontal>
-                            <samples>20</samples>
-                            <resolution>1</resolution>
-                            <min_angle>${-pi/90}</min_angle>
-                            <max_angle>${pi/90}</max_angle>
-                        </horizontal>
-                        <vertical>
-                            <samples>20</samples>
-                            <resolution>1</resolution>
-                            <min_angle>${-pi/150}</min_angle>
-                            <max_angle>${pi/150}</max_angle>
-                        </vertical>
-                    </scan>
-                    <range>
-                        <min>${min_range}</min>
-                        <max>${max_range}</max>
-                        <resolution>${resolution}</resolution>
-                    </range>
-                </ray>
-                <plugin name="${base_name}_plugin" filename="libgazebo_ros_ray_sensor.so">
-                    <ros>
-                        <namespace>${base_name}</namespace>
-                        <remapping>~/out:=range</remapping>
-                    </ros>
-                    <output_type>sensor_msgs/Range</output_type>
-                    <radiation_type>ultrasound</radiation_type>
-                    <frame_name>${base_name}</frame_name>
-                </plugin>
-            </sensor>
-        </gazebo>
     </xacro:macro>
 </robot>
