Commit message: update description

File: mobo_bot_description/urdf/controllers/gazebo_control.xacro (robot description, xacro)
@@ -20,10 +20,8 @@
             <odometry_topic>odom</odometry_topic>
             <odometry_frame>odom</odometry_frame>
-            <!-- <odometry_source>1</odometry_source> -->
             <robot_base_frame>base_link</robot_base_frame>
-            <ros>
-                <!-- <namespace>/br</namespace> -->
+            <!-- <ros>
                 <remapping>odom:=wheel/odometry</remapping>
-            </ros>
+            </ros> -->
         </plugin>
     </gazebo>

File: mobo_bot_description/urdf/robot_core.xacro (robot description, xacro)
@@ -151,4 +151,109 @@
     </xacro:if>
     <!--  ########################### -->
+     <!--  lidar -->
+    <xacro:property name="lidar_z_offset" value="0.04"/>
+    <xacro:insert_lidar
+        base_name="lidar"
+        parent_name="chassis"
+        x="0.01" y="0" z="${chassis_height+lidar_z_offset}"
+        mass="0.1" color="grey"/>
+    <xacro:if value="$(arg use_simulation)">
+        <gazebo reference="right_rim">
+            <material>Gazebo/Red</material>
+        </gazebo>
+    </xacro:if>
+    <gazebo reference="lidar">
+        <material>Gazebo/DarkGrey</material>
+        <sensor name="lidar" type="ray">
+            <pose> 0 0 0 0 0 0 </pose>
+            <visualize>false</visualize>
+            <update_rate>10</update_rate>
+            <ray>
+                <scan>
+                    <horizontal>
+                        <samples>360</samples>
+                        <min_angle>${-pi*2}</min_angle>
+                        <max_angle>${pi*2}</max_angle>
+                    </horizontal>
+                </scan>
+                <range>
+                    <min>0.1</min>
+                    <max>10.0</max>
+                </range>
+            </ray>
+            <plugin name="lidar_plugin" filename="libgazebo_ros_ray_sensor.so">
+                <ros>
+                    <namespace>lidar</namespace>
+                    <remapping>~/out:=scan</remapping>
+                </ros>
+                <output_type>sensor_msgs/LaserScan</output_type>
+                <frame_name>lidar</frame_name>
+            </plugin>
+        </sensor>
+    </gazebo>
+    <!--  imu -->
+    <xacro:insert_imu
+        base_name="imu"
+        parent_name="chassis"
+        x="0" y="0" z="${chassis_height}"/>
+    <!-- <xacro:if value="$(arg use_simulation)">
+        <gazebo reference="imu">
+            <sensor name="imu" type="imu">
+                <always_on>true</always_on>
+                <update_rate>20</update_rate>
+                <visualize>true</visualize>
+                <imu>
+                    <angular_velocity>
+                        <x>
+                            <noise type="gaussian">
+                                <mean>0.0</mean>
+                                <stddev>2e-4</stddev>
+                            </noise>
+                        </x>
+                        <y>
+                            <noise type="gaussian">
+                                <mean>0.0</mean>
+                                <stddev>2e-4</stddev>
+                            </noise>
+                        </y>
+                        <z>
+                            <noise type="gaussian">
+                                <mean>0.0</mean>
+                                <stddev>2e-4</stddev>
+                            </noise>
+                        </z>
+                    </angular_velocity>
+                    <linear_acceleration>
+                        <x>
+                            <noise type="gaussian">
+                                <mean>0.0</mean>
+                                <stddev>1.7e-2</stddev>
+                            </noise>
+                        </x>
+                        <y>
+                            <noise type="gaussian">
+                                <mean>0.0</mean>
+                                <stddev>1.7e-2</stddev>
+                            </noise>
+                        </y>
+                        <z>
+                            <noise type="gaussian">
+                                <mean>0.0</mean>
+                                <stddev>1.7e-2</stddev>
+                            </noise>
+                        </z>
+                    </linear_acceleration>
+                </imu>
+                <plugin name="imu_plugin" filename="libgazebo_ros_imu_sensor.so">
+                    <ros>
+                        <namespace>imu</namespace>
+                        <remapping>~/out:=data</remapping>
+                    </ros>
+                    <initial_orientation_as_reference>false</initial_orientation_as_reference>
+                    <frame_name>imu</frame_name>
+                </plugin>
+            </sensor>
+        </gazebo>
+    </xacro:if> -->
     <!--  sonar -->
     <xacro:insert_sonar
@@ -198,109 +303,4 @@
         </gazebo>
     </xacro:if> -->
-     <!--  lidar -->
-    <xacro:property name="lidar_z_offset" value="0.04"/>
-    <xacro:insert_lidar
-        base_name="lidar"
-        parent_name="chassis"
-        x="0.01" y="0" z="${chassis_height+lidar_z_offset}"
-        mass="0.1" color="grey"/>
-    <xacro:if value="$(arg use_simulation)">
-        <gazebo reference="right_rim">
-            <material>Gazebo/Red</material>
-        </gazebo>
-    </xacro:if>
-    <gazebo reference="lidar">
-        <material>Gazebo/DarkGrey</material>
-        <sensor name="lidar" type="ray">
-            <pose> 0 0 0 0 0 0 </pose>
-            <visualize>false</visualize>
-            <update_rate>10</update_rate>
-            <ray>
-                <scan>
-                    <horizontal>
-                        <samples>360</samples>
-                        <min_angle>${-pi*2}</min_angle>
-                        <max_angle>${pi*2}</max_angle>
-                    </horizontal>
-                </scan>
-                <range>
-                    <min>0.1</min>
-                    <max>10.0</max>
-                </range>
-            </ray>
-            <plugin name="lidar_plugin" filename="libgazebo_ros_ray_sensor.so">
-                <ros>
-                    <namespace>lidar</namespace>
-                    <remapping>~/out:=scan</remapping>
-                </ros>
-                <output_type>sensor_msgs/LaserScan</output_type>
-                <frame_name>lidar</frame_name>
-            </plugin>
-        </sensor>
-    </gazebo>
-    <!--  imu -->
-    <xacro:insert_imu
-        base_name="imu"
-        parent_name="chassis"
-        x="0" y="0" z="${chassis_height}"/>
-    <xacro:if value="$(arg use_simulation)">
-        <gazebo reference="imu">
-            <sensor name="imu" type="imu">
-                <always_on>true</always_on>
-                <update_rate>20</update_rate>
-                <visualize>true</visualize>
-                <imu>
-                    <angular_velocity>
-                        <x>
-                            <noise type="gaussian">
-                                <mean>0.0</mean>
-                                <stddev>2e-4</stddev>
-                            </noise>
-                        </x>
-                        <y>
-                            <noise type="gaussian">
-                                <mean>0.0</mean>
-                                <stddev>2e-4</stddev>
-                            </noise>
-                        </y>
-                        <z>
-                            <noise type="gaussian">
-                                <mean>0.0</mean>
-                                <stddev>2e-4</stddev>
-                            </noise>
-                        </z>
-                    </angular_velocity>
-                    <linear_acceleration>
-                        <x>
-                            <noise type="gaussian">
-                                <mean>0.0</mean>
-                                <stddev>1.7e-2</stddev>
-                            </noise>
-                        </x>
-                        <y>
-                            <noise type="gaussian">
-                                <mean>0.0</mean>
-                                <stddev>1.7e-2</stddev>
-                            </noise>
-                        </y>
-                        <z>
-                            <noise type="gaussian">
-                                <mean>0.0</mean>
-                                <stddev>1.7e-2</stddev>
-                            </noise>
-                        </z>
-                    </linear_acceleration>
-                </imu>
-                <plugin name="imu_plugin" filename="libgazebo_ros_imu_sensor.so">
-                    <ros>
-                        <namespace>imu</namespace>
-                        <remapping>~/out:=data</remapping>
-                    </ros>
-                    <initial_orientation_as_reference>false</initial_orientation_as_reference>
-                    <frame_name>imu</frame_name>
-                </plugin>
-            </sensor>
-        </gazebo>
-    </xacro:if>
     <!-- camera -->
     <!-- <xacro:property name="cam_x_offset" value="0.015"/>
@@ -310,6 +310,6 @@
         parent_name="chassis"
         x="${0.08+cam_x_offset}" y="0" z="${chassis_height+cam_z_offset}"
-        mass="0.005" tilt_angle="0" color="grey"/>
-    <xacro:if value="$(arg use_simulation)">
+        mass="0.005" tilt_angle="0" color="grey"/> -->
+    <!-- <xacro:if value="$(arg use_simulation)">
         <gazebo reference="camera">
           <material>Gazebo/DarkGrey</material>

Commit message: added igition sim successfully with EKF

File: mobo_bot_description/urdf/controllers/gazebo_control.xacro (robot description, xacro)
@@ -1,39 +1,29 @@
 <?xml version="1.0"?>
 <robot xmlns:xacro="http://ros.org/wiki/xacro">
-    <gazebo>
-        <plugin name="mobo_bot_diff_drive_gazebo_control" filename="libgazebo_ros_diff_drive.so">
-            <update_rate>40</update_rate>
-            <!-- wheels -->
-            <left_joint>left_wheel_joint</left_joint>
-            <right_joint>right_wheel_joint</right_joint>
-            <!-- kinematics -->
-            <wheel_separation>0.25</wheel_separation>
-            <wheel_diameter>0.068</wheel_diameter>
-            <!-- limits -->
-            <max_wheel_torque>20</max_wheel_torque>
-            <max_wheel_acceleration>2.0</max_wheel_acceleration>
-            <command_topic>cmd_vel</command_topic>
-            <!-- output -->
-            <publish_odom>true</publish_odom>
-            <publish_odom_tf>true</publish_odom_tf>
-            <publish_wheel_tf>true</publish_wheel_tf>
-            <odometry_topic>odom</odometry_topic>
-            <odometry_frame>odom</odometry_frame>
-            <robot_base_frame>base_link</robot_base_frame>
-            <!-- <ros>
-                <remapping>odom:=wheel/odometry</remapping>
-            </ros> -->
-        </plugin>
-    </gazebo>
-    <gazebo>
-        <plugin name="mobo_bot_joint_states" filename="libgazebo_ros_joint_state_publisher.so">
-            <ros>
-                <!-- <namespace>/br</namespace> -->
-                <remapping>~/out:=joint_states</remapping>
-            </ros>
-            <update_rate>30</update_rate>
-            <joint_name>left_wheel_joint</joint_name>
-            <joint_name>right_wheel_joint</joint_name>
-        </plugin>
-    </gazebo>
+    <ros2_control name="IgnitionSystem" type="system">
+    <hardware>
+      <plugin>ign_ros2_control/IgnitionSystem</plugin>
+    </hardware>
+    <joint name="left_wheel_joint">
+        <command_interface name="velocity">
+            <param name="min">-8.0</param>
+            <param name="max">8.0</param>
+        </command_interface>
+        <state_interface name="position"/>
+        <state_interface name="velocity"/>
+      </joint>
+      <joint name="right_wheel_joint">
+        <command_interface name="velocity">
+            <param name="min">-8.0</param>
+            <param name="max">8.0</param>
+        </command_interface>
+        <state_interface name="position"/>
+        <state_interface name="velocity"/>
+      </joint>
+  </ros2_control>
+  <gazebo>
+    <plugin filename="ign_ros2_control-system" name="ign_ros2_control::IgnitionROS2ControlPlugin">
+      <parameters>$(find mobo_bot_sim)/config/diff_drive_controller.yaml</parameters>
+    </plugin>
+  </gazebo>
 </robot>

File: mobo_bot_description/urdf/other_parts/box_with_fillet_macro.xacro (robot description, xacro)
@@ -1,5 +1,5 @@
 <?xml version="1.0"?>
 <robot xmlns:xacro="http://www.ros.org/wiki/xacro" >
-    <xacro:macro name="insert_box_with_fillet" params="x y z size_x size_y size_z fillet_radius color">
+    <xacro:macro name="insert_box_with_fillet" params="x y z size_x size_y size_z fillet_radius">
             <!-- logitudinal box -->
             <visual>
@@ -8,5 +8,7 @@
                     <box size="${size_x} ${size_y-(2*fillet_radius)} ${size_z}"/>
                 </geometry>
-                <material name="${color}"/>
+                <material name="DarkBlue">
+                  <color rgba="0.09 0.30 0.46 1.0"/>
+                </material>
             </visual>
             <!-- lateral box -->
@@ -16,5 +18,7 @@
                     <box size="${size_x-(2*fillet_radius)} ${size_y} ${size_z}"/>
                 </geometry>
-                <material name="${color}"/>
+                <material name="DarkBlue">
+                  <color rgba="0.09 0.30 0.46 1.0"/>
+                </material>
             </visual>
             <!-- cylinder1 -->
@@ -24,5 +28,7 @@
                     <cylinder length="${size_z}" radius="${fillet_radius}"/>
                 </geometry>
-                <material name="${color}"/>
+                <material name="DarkBlue">
+                  <color rgba="0.09 0.30 0.46 1.0"/>
+                </material>
             </visual>
             <!-- cylinder2 -->
@@ -32,5 +38,7 @@
                     <cylinder length="${size_z}" radius="${fillet_radius}"/>
                 </geometry>
-                <material name="${color}"/>
+                <material name="DarkBlue">
+                  <color rgba="0.09 0.30 0.46 1.0"/>
+                </material>
             </visual>
             <!-- cylinder3 -->
@@ -40,5 +48,7 @@
                     <cylinder length="${size_z}" radius="${fillet_radius}"/>
                 </geometry>
-                <material name="${color}"/>
+                <material name="DarkBlue">
+                  <color rgba="0.09 0.30 0.46 1.0"/>
+                </material>
             </visual>
             <!-- cylinder4 -->
@@ -48,5 +58,7 @@
                     <cylinder length="${size_z}" radius="${fillet_radius}"/>
                 </geometry>
-                <material name="${color}"/>
+                <material name="DarkBlue">
+                  <color rgba="0.09 0.30 0.46 1.0"/>
+                </material>
             </visual>
     </xacro:macro>

File: mobo_bot_description/urdf/other_parts/drive_wheel_macro.xacro (robot description, xacro)
@@ -15,5 +15,5 @@
         </inertial>
     </xacro:macro>
-    <xacro:macro name="insert_drive_wheel" params="base_name parent_name x y z mass radius thickness color">
+    <xacro:macro name="insert_drive_wheel" params="base_name parent_name x y z mass radius thickness">
         <joint name="${base_name}_joint" type="continuous">
             <parent link="${parent_name}"/>
@@ -21,4 +21,5 @@
             <origin xyz="${x} ${y} ${z}" rpy="${-pi/2} 0 0"/>
             <axis xyz="0 0 1"/>
+            <dynamics damping="0.2"/>
         </joint>
         <link name="${base_name}">
@@ -28,5 +29,7 @@
                     <cylinder radius="${radius}" length="${thickness}"/>
                 </geometry>
-                <material name="${color}"/>
+                <material name="black">
+                    <color rgba="0.1 0.1 0.1 1"/>
+                </material>
             </visual>
             <collision>

File: mobo_bot_description/urdf/other_parts/drive_wheel_rim_macro.xacro (robot description, xacro)
@@ -1,5 +1,5 @@
 <?xml version="1.0"?>
 <robot xmlns:xacro="http://www.ros.org/wiki/xacro" >
-    <xacro:macro name="insert_drive_wheel_rim" params="base_name parent_name radius thickness spoke_width color">
+    <xacro:macro name="insert_drive_wheel_rim" params="base_name parent_name radius thickness spoke_width">
         <joint name="${base_name}_joint" type="fixed">
             <parent link="${parent_name}"/>
@@ -13,5 +13,7 @@
                     <box size="${spoke_width} ${radius*1.3} ${thickness+0.001}"/>
                 </geometry>
-                <material name="${color}"/>
+                <material name="red">
+                    <color rgba="1 0.1 0.1 1"/>
+                </material>
             </visual>
             <visual>
@@ -20,5 +22,7 @@
                     <box size="${spoke_width} ${radius*1.3} ${thickness+0.001}"/>
                 </geometry>
-                <material name="${color}"/>
+                <material name="red">
+                    <color rgba="1 0.1 0.1 1"/>
+                </material>
             </visual>
             <visual>
@@ -27,5 +31,7 @@
                     <box size="${spoke_width} ${radius*1.3} ${thickness+0.001}"/>
                 </geometry>
-                <material name="${color}"/>
+                <material name="red">
+                    <color rgba="1 0.1 0.1 1"/>
+                </material>
             </visual>
             <visual>
@@ -34,5 +40,7 @@
                     <box size="${spoke_width} ${radius*1.3} ${thickness+0.001}"/>
                 </geometry>
-                <material name="${color}"/>
+                <material name="red">
+                    <color rgba="1 0.1 0.1 1"/>
+                </material>
             </visual>
         </link>
