Commit message: added igition sim successfully with EKF

File: mobo_bot_description/urdf/robot_core.xacro (robot description, xacro)
@@ -34,8 +34,8 @@
         <xacro:insert_box_with_fillet x="-0.025" y="0" z="0"
             size_x="${chassis_length}" size_y="${chassis_width}" size_z="${slab_height}"
-            fillet_radius="0.04" color="${chassis_color}"/>
+            fillet_radius="0.04"/>
         <xacro:insert_box_with_fillet x="-0.025" y="0" z="${chassis_height}"
             size_x="${chassis_length}" size_y="${chassis_width}" size_z="${slab_height}"
-            fillet_radius="0.04" color="${chassis_color}"/>
+            fillet_radius="0.04"/>
         <visual>
             <origin xyz="0.05 0.08 ${chassis_height/2}" rpy="0 0 0"/>
@@ -43,5 +43,7 @@
                 <cylinder radius="0.005" length="${chassis_height}"/>
             </geometry>
-            <material name="${chassis_color}"/>
+            <material name="DarkBlue">
+              <color rgba="0.09 0.30 0.46 1.0"/>
+            </material>
         </visual>
         <visual>
@@ -50,5 +52,7 @@
                 <cylinder radius="0.005" length="${chassis_height}"/>
             </geometry>
-            <material name="${chassis_color}"/>
+            <material name="DarkBlue">
+              <color rgba="0.09 0.30 0.46 1.0"/>
+            </material>
         </visual>
         <visual>
@@ -57,5 +61,7 @@
                 <cylinder radius="0.005" length="${chassis_height}"/>
             </geometry>
-            <material name="${chassis_color}"/>
+            <material name="DarkBlue">
+              <color rgba="0.09 0.30 0.46 1.0"/>
+            </material>
         </visual>
         <visual>
@@ -64,5 +70,7 @@
                 <cylinder radius="0.005" length="${chassis_height}"/>
             </geometry>
-            <material name="${chassis_color}"/>
+            <material name="DarkBlue">
+              <color rgba="0.09 0.30 0.46 1.0"/>
+            </material>
         </visual>
         <collision>
@@ -76,9 +84,4 @@
         </xacro:inertial_box>
     </link>
-    <xacro:if value="$(arg use_simulation)">
-        <gazebo reference="chassis">
-            <material>Gazebo/Orange</material>
-        </gazebo>
-    </xacro:if>
     <!--  ########################### -->
     <!-- LEFT DRIVE WHEEL -->
@@ -89,15 +92,9 @@
         mass="${wheel_mass}"
         radius="${wheel_radius}"
-        thickness="${wheel_width}"
-        color="black"/>
+        thickness="${wheel_width}"/>
     <xacro:if value="$(arg use_simulation)">
         <gazebo reference="left_wheel">
             <mu1>1.0</mu1>
             <mu2>1.0</mu2>
-            <!-- <kp>1000000</kp> -->
-            <!-- <kd>0.001</kd> -->
-            <minDepth>0.005</minDepth>
-            <!-- <fdir1>${fdir}</fdir1> -->
-            <material>Gazebo/FlatBlack</material>
         </gazebo>
     </xacro:if>
@@ -107,11 +104,5 @@
         radius="${wheel_radius}"
         thickness="${wheel_width}"
-        spoke_width="0.005"
-        color="red"/>
-    <xacro:if value="$(arg use_simulation)">
-        <gazebo reference="left_rim">
-            <material>Gazebo/Red</material>
-        </gazebo>
-    </xacro:if>
+        spoke_width="0.005"/>
     <!-- ############################# -->
     <!-- RIGHT DRIVE WHEEL -->
@@ -122,15 +113,9 @@
         mass="${wheel_mass}"
         radius="${wheel_radius}"
-        thickness="${wheel_width}"
-        color="black"/>
+        thickness="${wheel_width}"/>
     <xacro:if value="$(arg use_simulation)">
         <gazebo reference="right_wheel">
             <mu1>1.0</mu1>
             <mu2>1.0</mu2>
-            <!-- <kp>1000000</kp> -->
-            <!-- <kd>0.001</kd> -->
-            <minDepth>0.005</minDepth>
-            <!-- <fdir1>${fdir}</fdir1> -->
-            <material>Gazebo/FlatBlack</material>
         </gazebo>
     </xacro:if>
@@ -140,11 +125,5 @@
         radius="${wheel_radius}"
         thickness="${wheel_width}"
-        spoke_width="0.005"
-        color="red"/>
-    <xacro:if value="$(arg use_simulation)">
-        <gazebo reference="right_rim">
-            <material>Gazebo/Red</material>
-        </gazebo>
-    </xacro:if>
+        spoke_width="0.005"/>
     <!-- ############################# -->
     <!--  castor WHEEL LINK -->
@@ -160,5 +139,7 @@
                 <sphere radius="${castor_wheel_radius/2}" />
             </geometry>
-            <material name="grey"/>
+            <material name="grey">
+                <color rgba="0.25 0.25 0.25 1"/>
+            </material>
         </visual>
         <collision>
@@ -176,9 +157,4 @@
             <mu1>0.001</mu1>
             <mu2>0.001</mu2>
-            <!-- <kp>1000000.0</kp> -->
-            <!-- <kd>1.0</kd> -->
-            <!-- <fdir1>1 0 0</fdir1> -->
-            <!-- <minDepth>0.01</minDepth> -->
-            <material>Gazebo/Grey</material>
         </gazebo>
     </xacro:if>
@@ -190,37 +166,27 @@
         parent_name="chassis"
         x="0.01" y="0" z="${chassis_height+lidar_z_offset}"
-        mass="0.1" color="grey"/>
-    <xacro:if value="$(arg use_simulation)">
-        <gazebo reference="lidar">
-            <material>Gazebo/DarkGrey</material>
-        </gazebo>
-    </xacro:if>
+        mass="0.1"/>
     <xacro:if value="$(arg use_simulation)">
       <gazebo reference="lidar">
-        <sensor name="lidar" type="ray">
-            <pose> 0 0 0 0 0 0 </pose>
-            <visualize>false</visualize>
-            <update_rate>10</update_rate>
-            <ray>
-                <scan>
-                    <horizontal>
-                        <samples>360</samples>
-                        <min_angle>${-pi*2}</min_angle>
-                        <max_angle>${pi*2}</max_angle>
-                    </horizontal>
-                </scan>
-                <range>
-                    <min>0.1</min>
-                    <max>10.0</max>
-                </range>
-            </ray>
-            <plugin name="lidar_plugin" filename="libgazebo_ros_ray_sensor.so">
-                <ros>
-                    <namespace>lidar</namespace>
-                    <remapping>~/out:=scan</remapping>
-                </ros>
-                <output_type>sensor_msgs/LaserScan</output_type>
-                <frame_name>lidar</frame_name>
-            </plugin>
+        <sensor name="lidar" type="gpu_lidar">
+          <pose> 0 0 0 0 0 0 </pose>
+          <ignition_frame_id>lidar</ignition_frame_id>
+          <topic>lidar/scan</topic>
+          <always_on>true</always_on>
+          <visualize>true</visualize>
+          <update_rate>10</update_rate>
+          <ray>
+            <scan>
+                <horizontal>
+                    <samples>360</samples>
+                    <min_angle>${-pi*2}</min_angle>
+                    <max_angle>${pi*2}</max_angle>
+                </horizontal>
+            </scan>
+            <range>
+                <min>0.1</min>
+                <max>10.0</max>
+            </range>
+          </ray>
         </sensor>
       </gazebo>
@@ -231,63 +197,71 @@
         parent_name="chassis"
         x="0" y="0" z="${chassis_height}"/>
-    <!-- <xacro:if value="$(arg use_simulation)">
-        <gazebo reference="imu">
+    <xacro:if value="$(arg use_simulation)">
+          <gazebo reference="imu">
             <sensor name="imu" type="imu">
-                <always_on>true</always_on>
-                <update_rate>20</update_rate>
-                <visualize>true</visualize>
-                <imu>
-                    <angular_velocity>
-                        <x>
-                            <noise type="gaussian">
-                                <mean>0.0</mean>
-                                <stddev>2e-4</stddev>
-                            </noise>
-                        </x>
-                        <y>
-                            <noise type="gaussian">
-                                <mean>0.0</mean>
-                                <stddev>2e-4</stddev>
-                            </noise>
-                        </y>
-                        <z>
-                            <noise type="gaussian">
-                                <mean>0.0</mean>
-                                <stddev>2e-4</stddev>
-                            </noise>
-                        </z>
-                    </angular_velocity>
-                    <linear_acceleration>
-                        <x>
-                            <noise type="gaussian">
-                                <mean>0.0</mean>
-                                <stddev>1.7e-2</stddev>
-                            </noise>
-                        </x>
-                        <y>
-                            <noise type="gaussian">
-                                <mean>0.0</mean>
-                                <stddev>1.7e-2</stddev>
-                            </noise>
-                        </y>
-                        <z>
-                            <noise type="gaussian">
-                                <mean>0.0</mean>
-                                <stddev>1.7e-2</stddev>
-                            </noise>
-                        </z>
-                    </linear_acceleration>
-                </imu>
-                <plugin name="imu_plugin" filename="libgazebo_ros_imu_sensor.so">
-                    <ros>
-                        <namespace>imu</namespace>
-                        <remapping>~/out:=data</remapping>
-                    </ros>
-                    <initial_orientation_as_reference>false</initial_orientation_as_reference>
-                    <frame_name>imu</frame_name>
-                </plugin>
+              <ignition_frame_id>imu</ignition_frame_id>
+              <plugin filename="ignition-gazebo-imu-system" name="ignition::gazebo::systems::Imu">
+              </plugin>
+              <topic>imu/data</topic>
+              <always_on>true</always_on>
+              <update_rate>10</update_rate>
+              <visualize>true</visualize>
+              <imu>
+                <angular_velocity>
+                  <x>
+                    <noise type="gaussian">
+                      <mean>0.0</mean>
+                      <stddev>2e-4</stddev>
+                      <bias_mean>0.0000075</bias_mean>
+                      <bias_stddev>0.0000008</bias_stddev>
+                    </noise>
+                  </x>
+                  <y>
+                    <noise type="gaussian">
+                      <mean>0.0</mean>
+                      <stddev>2e-4</stddev>
+                      <bias_mean>0.0000075</bias_mean>
+                      <bias_stddev>0.0000008</bias_stddev>
+                    </noise>
+                  </y>
+                  <z>
+                    <noise type="gaussian">
+                      <mean>0.0</mean>
+                      <stddev>2e-4</stddev>
+                      <bias_mean>0.0000075</bias_mean>
+                      <bias_stddev>0.0000008</bias_stddev>
+                    </noise>
+                  </z>
+                </angular_velocity>
+                <linear_acceleration>
+                  <x>
+                    <noise type="gaussian">
+                      <mean>0.0</mean>
+                      <stddev>1.7e-2</stddev>
+                      <bias_mean>0.1</bias_mean>
+                      <bias_stddev>0.001</bias_stddev>
+                    </noise>
+                  </x>
+                  <y>
+                    <noise type="gaussian">
+                      <mean>0.0</mean>
+                      <stddev>1.7e-2</stddev>
+                      <bias_mean>0.1</bias_mean>
+                      <bias_stddev>0.001</bias_stddev>
+                    </noise>
+                  </y>
+                  <z>
+                    <noise type="gaussian">
+                      <mean>0.0</mean>
+                      <stddev>1.7e-2</stddev>
+                      <bias_mean>0.1</bias_mean>
+                      <bias_stddev>0.001</bias_stddev>
+                    </noise>
+                  </z>
+                </linear_acceleration>
+              </imu>
             </sensor>
         </gazebo>
-    </xacro:if> -->
+    </xacro:if>
     <!--  sonar -->
     <xacro:insert_sonar
@@ -295,50 +269,5 @@
         parent_name="chassis"
         x="0.0825" y="0" z="${chassis_height/6}"
-        mass="0.005" color="blue"/>
-    <xacro:if value="$(arg use_simulation)">
-        <gazebo reference="sonar">
-            <material>Gazebo/Blue</material>
-        </gazebo>
-    </xacro:if>
-    <!-- <xacro:if value="$(arg use_simulation)">
-          <gazebo reference="sonar">
-            <sensor name="sonar" type="ray">
-                <always_on>false</always_on>
-                <visualize>false</visualize>
-                <pose>0.0 0 0.0 0 0 0</pose>
-                <update_rate>10</update_rate>
-                <ray>
-                    <scan>
-                        <horizontal>
-                            <samples>20</samples>
-                            <resolution>1</resolution>
-                            <min_angle>${-pi/90}</min_angle>
-                            <max_angle>${pi/90}</max_angle>
-                        </horizontal>
-                        <vertical>
-                            <samples>20</samples>
-                            <resolution>1</resolution>
-                            <min_angle>${-pi/150}</min_angle>
-                            <max_angle>${pi/150}</max_angle>
-                        </vertical>
-                    </scan>
-                    <range>
-                        <min>0.01</min>
-                        <max>4.0</max>
-                        <resolution>0.01</resolution>
-                    </range>
-                </ray>
-                <plugin name="sonar_plugin" filename="libgazebo_ros_ray_sensor.so">
-                    <ros>
-                        <namespace>sonar</namespace>
-                        <remapping>~/out:=range</remapping>
-                    </ros>
-                    <output_type>sensor_msgs/Range</output_type>
-                    <radiation_type>ultrasound</radiation_type>
-                    <frame_name>sonar</frame_name>
-                </plugin>
-            </sensor>
-        </gazebo>
-    </xacro:if> -->
+        mass="0.005"/>
     <!-- camera -->
     <xacro:property name="cam_x_offset" value="0.015"/>
@@ -348,31 +277,25 @@
         parent_name="chassis"
         x="${0.08+cam_x_offset}" y="0" z="${chassis_height}"
-        mass="0.005" tilt_angle="0.00" color="grey"/>
-    <xacro:if value="$(arg use_simulation)">
-        <gazebo reference="camera">
-            <material>Gazebo/DarkGrey</material>
-        </gazebo>
-    </xacro:if>
+        mass="0.005" tilt_angle="0.00"/>
+    <!-- <ignition_frame_id>camera_optical_link</ignition_frame_id> -->
     <!-- <xacro:if value="$(arg use_simulation)">
-        <gazebo reference="camera">
+        <gazebo reference="camera_optical_link">
           <sensor name="camera" type="camera">
-            <pose> 0 0 0 0 0 0 </pose>
-            <visualize>false</visualize>
-            <update_rate>20</update_rate>
             <camera>
-                <horizontal_fov>1.46608</horizontal_fov>
-                <image>
-                    <format>R8G8B8</format>
-                    <width>320</width>
-                    <height>240</height>
-                </image>
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
File: mobo_bot_description/urdf/robot_urdf.xacro (robot description, xacro)
@@ -8,5 +8,5 @@
     <!-- <xacro:arg name="cam_visual"   default="false"/> -->
     <!-- ############################################### -->
-    <xacro:include filename="$(find mobo_bot_description)/urdf/color_macros.xacro" />
+    <!-- <xacro:include filename="$(find mobo_bot_description)/urdf/color_macros.xacro" /> -->
     <xacro:include filename="$(find mobo_bot_description)/urdf/inertia_macros.xacro" />
     <xacro:include filename="$(find mobo_bot_description)/urdf/robot_core.xacro" />

File: mobo_bot_description/urdf/sensors/cam.xacro (robot description, xacro)
@@ -1,5 +1,5 @@
 <?xml version="1.0"?>
 <robot xmlns:xacro="http://www.ros.org/wiki/xacro" >
-    <xacro:macro name="insert_camera" params="base_name parent_name x y z mass tilt_angle color">
+    <xacro:macro name="insert_camera" params="base_name parent_name x y z mass tilt_angle">
         <joint name="${base_name}_joint" type="fixed">
             <parent link="${parent_name}"/>
@@ -13,5 +13,7 @@
                     <cylinder radius="0.007" length="0.01"/>
                 </geometry>
-                <material name="${color}"/>
+                <material name="grey">
+                    <color rgba="0.25 0.25 0.25 1"/>
+                </material>
             </visual>
             <visual>
@@ -20,5 +22,7 @@
                     <box size="0.02 0.03 0.01"/>
                 </geometry>
-                <material name="${color}"/>
+                <material name="grey">
+                    <color rgba="0.25 0.25 0.25 1"/>
+                </material>
             </visual>
             <collision>
@@ -40,44 +44,2 @@
     </xacro:macro>
 </robot>
- <!-- <joint name="line_cam_joint" type="fixed">
-        <parent link="chassis"/>
-        <child link="line_cam"/>
-        <origin xyz="0.305 0 0.08" rpy="0 0 0"/>
-    </joint>
-    <link name="line_cam">
-        <visual>
-            <geometry>
-                <box size="0.010 0.03 0.03"/>
-            </geometry>
-            <material name="red"/>
-        </visual>
-    </link>
-    <joint name="line_cam_optical_joint" type="fixed">
-        <parent link="line_cam"/>
-        <child link="line_cam_link_optical"/>
-        <origin xyz="0 0 0" rpy="${-pi/2} 0 ${-pi/2}"/>
-    </joint>
-    <link name="line_cam_link_optical"></link>
-    <gazebo reference="line_cam">
-        <material>Gazebo/Red</material>
-        <sensor name="line_cam" type="camera">
-            <pose> 0 0 0 0 0 0 </pose>
-            <visualize>true</visualize>
-            <update_rate>10</update_rate>
-            <camera>
-                <horizontal_fov>1.089</horizontal_fov>
-                <image>
-                    <format>R8G8B8</format>
-                    <width>640</width>
-                    <height>480</height>
-                </image>
-                <clip>
-                    <near>0.05</near>
-                    <far>8.0</far>
-                </clip>
-            </camera>
-            <plugin name="camera_controller" filename="libgazebo_ros_camera.so">
-                <frame_name>line_cam_link_optical</frame_name>
-            </plugin>
-        </sensor>
-    </gazebo> -->

File: mobo_bot_description/urdf/sensors/lidar.xacro (robot description, xacro)
@@ -1,5 +1,5 @@
 <?xml version="1.0"?>
 <robot xmlns:xacro="http://www.ros.org/wiki/xacro" >
-    <xacro:macro name="insert_lidar" params="base_name parent_name x y z mass color">
+    <xacro:macro name="insert_lidar" params="base_name parent_name x y z mass">
         <joint name="${base_name}_joint" type="fixed">
             <parent link="${parent_name}"/>
@@ -13,5 +13,7 @@
                     <cylinder radius="0.03" length="0.04"/>
                 </geometry>
-                <material name="${color}"/>
+                <material name="grey">
+                    <color rgba="0.25 0.25 0.25 1"/>
+                </material>
             </visual>
             <collision>

File: mobo_bot_description/urdf/sensors/sonar.xacro (robot description, xacro)
@@ -4,5 +4,5 @@
     <!-- <xacro:property name="deg2rad" value="0.017460317"/>
     <xacro:property name="scan_angle" value="1"/> -->
-    <xacro:macro name="insert_sonar" params="base_name parent_name x y z mass color">
+    <xacro:macro name="insert_sonar" params="base_name parent_name x y z mass">
         <joint name="${base_name}_joint" type="fixed">
             <parent link="${parent_name}"/>
@@ -16,5 +16,7 @@
                     <cylinder radius="0.006" length="0.006"/>
                 </geometry>
-                <material name="${color}"/>
+                <material name="blue">
+                    <color rgba="0.2 0.2 1 1"/>
+                </material>
             </visual>
             <collision>
@@ -29,5 +31,7 @@
                     <cylinder radius="0.006" length="0.006"/>
                 </geometry>
-                <material name="${color}"/>
+                <material name="blue">
+                    <color rgba="0.2 0.2 1 1"/>
+                </material>
             </visual>
             <collision>
