Commit message: update base control codes

File: mobo_bot_description/urdf/controllers/epmc_ros2_control.xacro (robot description, xacro)
@@ -8,5 +8,5 @@
         <param name="motorB_wheel_name">right_wheel_joint</param>
         <!-- <param name="port">/dev/ttyUSB0</param> -->
-        <param name="port">/dev/serial/by-path/pci-0000:00:14.0-usb-0:1.4:1.0-port0</param>
+        <param name="port">/dev/serial/by-path/platform-fd500000.pcie-pci-0000:01:00.0-usb-0:1.1.4:1.0-port0</param>
         <param name="cmd_vel_timeout_ms">2000</param>
       </hardware>

File: mobo_bot_description/urdf/other_parts/box_with_fillet_macro.xacro (robot description, xacro)
@@ -8,6 +8,6 @@
                     <box size="${size_x} ${size_y-(2*fillet_radius)} ${size_z}"/>
                 </geometry>
-                <material name="DarkBlue">
-                  <color rgba="0.09 0.30 0.46 1.0"/>
+                <material name="orange">
+                  <color rgba="1 0.55 0 1"/>
                 </material>
             </visual>
@@ -18,6 +18,6 @@
                     <box size="${size_x-(2*fillet_radius)} ${size_y} ${size_z}"/>
                 </geometry>
-                <material name="DarkBlue">
-                  <color rgba="0.09 0.30 0.46 1.0"/>
+                <material name="orange">
+                  <color rgba="1 0.55 0 1"/>
                 </material>
             </visual>
@@ -28,6 +28,6 @@
                     <cylinder length="${size_z}" radius="${fillet_radius}"/>
                 </geometry>
-                <material name="DarkBlue">
-                  <color rgba="0.09 0.30 0.46 1.0"/>
+                <material name="orange">
+                  <color rgba="1 0.55 0 1"/>
                 </material>
             </visual>
@@ -38,6 +38,6 @@
                     <cylinder length="${size_z}" radius="${fillet_radius}"/>
                 </geometry>
-                <material name="DarkBlue">
-                  <color rgba="0.09 0.30 0.46 1.0"/>
+                <material name="orange">
+                  <color rgba="1 0.55 0 1"/>
                 </material>
             </visual>
@@ -48,6 +48,6 @@
                     <cylinder length="${size_z}" radius="${fillet_radius}"/>
                 </geometry>
-                <material name="DarkBlue">
-                  <color rgba="0.09 0.30 0.46 1.0"/>
+                <material name="orange">
+                  <color rgba="1 0.55 0 1"/>
                 </material>
             </visual>
@@ -58,6 +58,6 @@
                     <cylinder length="${size_z}" radius="${fillet_radius}"/>
                 </geometry>
-                <material name="DarkBlue">
-                  <color rgba="0.09 0.30 0.46 1.0"/>
+                <material name="orange">
+                  <color rgba="1 0.55 0 1"/>
                 </material>
             </visual>

File: mobo_bot_description/urdf/robot_core.xacro (robot description, xacro)
@@ -43,6 +43,6 @@
                 <cylinder radius="0.005" length="${chassis_height}"/>
             </geometry>
-            <material name="DarkBlue">
-              <color rgba="0.09 0.30 0.46 1.0"/>
+            <material name="orange">
+                <color rgba="1 0.55 0 1"/>
             </material>
         </visual>
@@ -52,6 +52,6 @@
                 <cylinder radius="0.005" length="${chassis_height}"/>
             </geometry>
-            <material name="DarkBlue">
-              <color rgba="0.09 0.30 0.46 1.0"/>
+            <material name="orange">
+                <color rgba="1 0.55 0 1"/>
             </material>
         </visual>
@@ -61,6 +61,6 @@
                 <cylinder radius="0.005" length="${chassis_height}"/>
             </geometry>
-            <material name="DarkBlue">
-              <color rgba="0.09 0.30 0.46 1.0"/>
+            <material name="orange">
+                <color rgba="1 0.55 0 1"/>
             </material>
         </visual>
@@ -70,6 +70,6 @@
                 <cylinder radius="0.005" length="${chassis_height}"/>
             </geometry>
-            <material name="DarkBlue">
-              <color rgba="0.09 0.30 0.46 1.0"/>
+            <material name="orange">
+                <color rgba="1 0.55 0 1"/>
             </material>
         </visual>

Commit message: pi-test

File: mobo_bot_description/urdf/controllers/epmc_ros2_control.xacro (robot description, xacro)
@@ -8,5 +8,5 @@
         <param name="motorB_wheel_name">right_wheel_joint</param>
         <!-- <param name="port">/dev/ttyUSB0</param> -->
-        <param name="port">/dev/serial/by-path/platform-fd500000.pcie-pci-0000:01:00.0-usb-0:1.1.4:1.0-port0</param>
+        <param name="port">/dev/serial/by-path/platform-fd500000.pcie-pci-0000:01:00.0-usb-0:1.2.4:1.0-port0</param>
         <param name="cmd_vel_timeout_ms">2000</param>
       </hardware>

File: mobo_bot_description/urdf/robot_core.xacro (robot description, xacro)
@@ -278,7 +278,7 @@
         x="${0.08+cam_x_offset}" y="0" z="${chassis_height}"
         mass="0.005" tilt_angle="0.00"/>
-    <!-- <ignition_frame_id>camera_optical_link</ignition_frame_id> -->
+    <!-- <ignition_frame_id>camera_optical</ignition_frame_id> -->
     <!-- <xacro:if value="$(arg use_simulation)">
-        <gazebo reference="camera_optical_link">
+        <gazebo reference="camera_optical">
           <sensor name="camera" type="camera">
             <camera>

File: mobo_bot_description/urdf/sensors/cam.xacro (robot description, xacro)
@@ -38,8 +38,8 @@
         <joint name="${base_name}_optical_joint" type="fixed">
             <parent link="${base_name}"/>
-            <child link="${base_name}_optical_link"/>
+            <child link="${base_name}_optical"/>
             <origin xyz="0 0 0" rpy="${-pi/2} 0 ${-pi/2}"/>
         </joint>
-        <link name="${base_name}_optical_link"/>
+        <link name="${base_name}_optical"/>
     </xacro:macro>
 </robot>

Commit message: cleaned urdf code

File: mobo_bot_description/urdf/controllers/epmc_ros2_control.xacro (robot description, xacro)
@@ -1,5 +1,4 @@
 <?xml version="1.0"?>
 <robot xmlns:xacro="http://www.ros.org/wiki/xacro">
-    <!-- ############# add ros2_control => INSERT EPMC_HARDWARE_INTERFACE ############### -->
     <ros2_control name="epmc_ros2_control" type="system">
       <hardware>
@@ -7,5 +6,4 @@
         <param name="motorA_wheel_name">left_wheel_joint</param>
         <param name="motorB_wheel_name">right_wheel_joint</param>
-        <!-- <param name="port">/dev/ttyUSB0</param> -->
         <param name="port">/dev/serial/by-path/platform-fd500000.pcie-pci-0000:01:00.0-usb-0:1.2.4:1.0-port0</param>
         <param name="cmd_vel_timeout_ms">2000</param>
@@ -13,6 +11,6 @@
       <joint name="left_wheel_joint">
         <command_interface name="velocity">
-            <param name="min">-8.0</param> <!-- rad/sec -->
-            <param name="max">8.0</param> <!-- rad/sec -->
+            <param name="min">-8.0</param>
+            <param name="max">8.0</param>
         </command_interface>
         <state_interface name="position"/>
@@ -21,6 +19,6 @@
       <joint name="right_wheel_joint">
         <command_interface name="velocity">
-            <param name="min">-8.0</param> <!-- rad/sec -->
-            <param name="max">8.0</param> <!-- rad/sec -->
+            <param name="min">-8.0</param>
+            <param name="max">8.0</param>
         </command_interface>
         <state_interface name="position"/>
@@ -28,4 +26,3 @@
       </joint>
     </ros2_control>
-    <!-- ################################################################# -->
 </robot>

File: mobo_bot_description/urdf/controllers/gazebo_control.xacro (robot description, xacro)
@@ -1,5 +1,5 @@
 <?xml version="1.0"?>
 <robot xmlns:xacro="http://ros.org/wiki/xacro">
-    <ros2_control name="IgnitionSystem" type="system">
+  <ros2_control name="IgnitionSystem" type="system">
     <hardware>
       <plugin>ign_ros2_control/IgnitionSystem</plugin>

File: mobo_bot_description/urdf/inertia_macros.xacro (robot description, xacro)
@@ -1,7 +1,4 @@
 <?xml version="1.0"?>
 <robot xmlns:xacro="http://www.ros.org/wiki/xacro" >
-    <!-- Specify some standard inertial calculations https://en.wikipedia.org/wiki/List_of_moments_of_inertia -->
-    <!-- These make use of xacro's mathematical functionality -->
-    <!-- ################### inertia macros  ############################-->
     <xacro:macro name="inertial_sphere" params="mass radius *origin">
         <inertial>
@@ -31,4 +28,3 @@
         </inertial>
     </xacro:macro>
-    <!-- ###################################################################################### -->
 </robot>

File: mobo_bot_description/urdf/other_parts/box_with_fillet_macro.xacro (robot description, xacro)
@@ -2,64 +2,58 @@
 <robot xmlns:xacro="http://www.ros.org/wiki/xacro" >
     <xacro:macro name="insert_box_with_fillet" params="x y z size_x size_y size_z fillet_radius">
-            <!-- logitudinal box -->
-            <visual>
-                <origin xyz="${x} ${y} ${z}" rpy="0 0 0"/>
-                <geometry>
-                    <box size="${size_x} ${size_y-(2*fillet_radius)} ${size_z}"/>
-                </geometry>
-                <material name="orange">
-                  <color rgba="1 0.55 0 1"/>
-                </material>
-            </visual>
-            <!-- lateral box -->
-            <visual>
-                <origin xyz="${x} ${y} ${z}" rpy="0 0 0"/>
-                <geometry>
-                    <box size="${size_x-(2*fillet_radius)} ${size_y} ${size_z}"/>
-                </geometry>
-                <material name="orange">
-                  <color rgba="1 0.55 0 1"/>
-                </material>
-            </visual>
-            <!-- cylinder1 -->
-            <visual>
-                <origin xyz="${x+((size_x/2)-fillet_radius)} ${y+((size_y/2)-fillet_radius)} ${z}" rpy="0 0 0"/>
-                <geometry>
-                    <cylinder length="${size_z}" radius="${fillet_radius}"/>
-                </geometry>
-                <material name="orange">
-                  <color rgba="1 0.55 0 1"/>
-                </material>
-            </visual>
-            <!-- cylinder2 -->
-            <visual>
-                <origin xyz="${x+((size_x/2)-fillet_radius)} ${y-((size_y/2)-fillet_radius)} ${z}" rpy="0 0 0"/>
-                <geometry>
-                    <cylinder length="${size_z}" radius="${fillet_radius}"/>
-                </geometry>
-                <material name="orange">
-                  <color rgba="1 0.55 0 1"/>
-                </material>
-            </visual>
-            <!-- cylinder3 -->
-            <visual>
-                <origin xyz="${x-((size_x/2)-fillet_radius)} ${y+((size_y/2)-fillet_radius)} ${z}" rpy="0 0 0"/>
-                <geometry>
-                    <cylinder length="${size_z}" radius="${fillet_radius}"/>
-                </geometry>
-                <material name="orange">
-                  <color rgba="1 0.55 0 1"/>
-                </material>
-            </visual>
-            <!-- cylinder4 -->
-            <visual>
-                <origin xyz="${x-((size_x/2)-fillet_radius)} ${y-((size_y/2)-fillet_radius)} ${z}" rpy="0 0 0"/>
-                <geometry>
-                    <cylinder length="${size_z}" radius="${fillet_radius}"/>
-                </geometry>
-                <material name="orange">
-                  <color rgba="1 0.55 0 1"/>
-                </material>
-            </visual>
+        <visual>
+            <origin xyz="${x} ${y} ${z}" rpy="0 0 0"/>
+            <geometry>
+                <box size="${size_x} ${size_y-(2*fillet_radius)} ${size_z}"/>
+            </geometry>
+            <material name="orange">
+              <color rgba="1 0.55 0 1"/>
+            </material>
+        </visual>
+        <visual>
+            <origin xyz="${x} ${y} ${z}" rpy="0 0 0"/>
+            <geometry>
+                <box size="${size_x-(2*fillet_radius)} ${size_y} ${size_z}"/>
+            </geometry>
+            <material name="orange">
+              <color rgba="1 0.55 0 1"/>
+            </material>
+        </visual>
+        <visual>
+            <origin xyz="${x+((size_x/2)-fillet_radius)} ${y+((size_y/2)-fillet_radius)} ${z}" rpy="0 0 0"/>
+            <geometry>
+                <cylinder length="${size_z}" radius="${fillet_radius}"/>
+            </geometry>
+            <material name="orange">
+              <color rgba="1 0.55 0 1"/>
+            </material>
+        </visual>
+        <visual>
+            <origin xyz="${x+((size_x/2)-fillet_radius)} ${y-((size_y/2)-fillet_radius)} ${z}" rpy="0 0 0"/>
+            <geometry>
+                <cylinder length="${size_z}" radius="${fillet_radius}"/>
+            </geometry>
+            <material name="orange">
+              <color rgba="1 0.55 0 1"/>
+            </material>
+        </visual>
+        <visual>
+            <origin xyz="${x-((size_x/2)-fillet_radius)} ${y+((size_y/2)-fillet_radius)} ${z}" rpy="0 0 0"/>
+            <geometry>
+                <cylinder length="${size_z}" radius="${fillet_radius}"/>
+            </geometry>
+            <material name="orange">
+              <color rgba="1 0.55 0 1"/>
+            </material>
+        </visual>
+        <visual>
+            <origin xyz="${x-((size_x/2)-fillet_radius)} ${y-((size_y/2)-fillet_radius)} ${z}" rpy="0 0 0"/>
+            <geometry>
+                <cylinder length="${size_z}" radius="${fillet_radius}"/>
+            </geometry>
+            <material name="orange">
+              <color rgba="1 0.55 0 1"/>
+            </material>
+        </visual>
     </xacro:macro>
 </robot>

File: mobo_bot_description/urdf/other_parts/drive_wheel_macro.xacro (robot description, xacro)
@@ -1,9 +1,4 @@
 <?xml version="1.0"?>
 <robot xmlns:xacro="http://www.ros.org/wiki/xacro" >
-    <xacro:macro name="material_black">
-        <material name="black">
-            <color rgba="0.1 0.1 0.1 1"/>
-        </material>
-    </xacro:macro>
     <xacro:macro name="inertial_cylinder" params="mass length radius *origin">
         <inertial>
@@ -37,5 +32,4 @@
                 <geometry>
                     <cylinder radius="${radius}" length="${thickness}"/>
-                    <!-- <sphere radius="${radius}"/> -->
                 </geometry>
             </collision>

File: mobo_bot_description/urdf/robot_core.xacro (robot description, xacro)
@@ -20,10 +20,6 @@
     <xacro:property name="castor_wheel_radius" value="${wheel_radius}"/>
     <xacro:property name="castor_wheel_mass" value="0.08"/>
-    <!-- BASE LINK -->
-    <!-- <base joint/> -->
     <link name="base_link">
     </link>
-    <!-- ################# -->
-    <!-- CHASSIS LINK -->
     <joint name="chassis_joint" type="fixed">
         <parent link="base_link"/>
@@ -84,6 +80,4 @@
         </xacro:inertial_box>
     </link>
-    <!--  ########################### -->
-    <!-- LEFT DRIVE WHEEL -->
     <xacro:insert_drive_wheel
         base_name="left_wheel"
@@ -105,6 +99,4 @@
         thickness="${wheel_width}"
         spoke_width="0.005"/>
-    <!-- ############################# -->
-    <!-- RIGHT DRIVE WHEEL -->
     <xacro:insert_drive_wheel
         base_name="right_wheel"
@@ -126,6 +118,4 @@
         thickness="${wheel_width}"
         spoke_width="0.005"/>
-    <!-- ############################# -->
-    <!--  castor WHEEL LINK -->
     <joint name="castor_wheel_joint" type="fixed">
         <parent link="base_link"/>
@@ -159,6 +149,4 @@
         </gazebo>
     </xacro:if>
-    <!--  ########################### -->
-     <!--  lidar -->
     <xacro:property name="lidar_z_offset" value="0.04"/>
     <xacro:insert_lidar
@@ -192,5 +180,4 @@
       </gazebo>
     </xacro:if>
-    <!--  imu -->
     <xacro:insert_imu
         base_name="imu"
@@ -264,5 +251,4 @@
         </gazebo>
     </xacro:if>
-    <!--  sonar -->
     <xacro:insert_sonar
         base_name="sonar"
@@ -270,5 +256,4 @@
         x="0.0825" y="0" z="${chassis_height/6}"
         mass="0.005"/>
-    <!-- camera -->
     <xacro:property name="cam_x_offset" value="0.015"/>
     <xacro:property name="cam_z_offset" value="0.01"/>
@@ -278,8 +263,8 @@
         x="${0.08+cam_x_offset}" y="0" z="${chassis_height}"
         mass="0.005" tilt_angle="0.00"/>
-    <!-- <ignition_frame_id>camera_optical</ignition_frame_id> -->
-    <!-- <xacro:if value="$(arg use_simulation)">
+    <xacro:if value="$(arg use_simulation)">
         <gazebo reference="camera_optical">
           <sensor name="camera" type="camera">
+            <ignition_frame_id>camera_optical</ignition_frame_id>
             <camera>
               <horizontal_fov>1.047</horizontal_fov>
@@ -300,4 +285,4 @@
           </sensor>
         </gazebo>
-    </xacro:if> -->
+    </xacro:if>
 </robot>

File: mobo_bot_description/urdf/robot_urdf.xacro (robot description, xacro)
@@ -1,12 +1,5 @@
 <?xml version="1.0"?>
 <robot name="mobo_bot" xmlns:xacro="http://www.ros.org/wiki/xacro">
-    <!-- ########### ARGUMENTS ######################### -->
     <xacro:arg name="use_simulation" default="false"/>
-    <!-- <xacro:arg name="laser_visual" default="false"/> -->
-    <!-- <xacro:arg name="imu_visual"   default="true"/> -->
-    <!-- <xacro:arg name="sonar_visual"   default="false"/> -->
-    <!-- <xacro:arg name="cam_visual"   default="false"/> -->
-    <!-- ############################################### -->
-    <!-- <xacro:include filename="$(find mobo_bot_description)/urdf/color_macros.xacro" /> -->
     <xacro:include filename="$(find mobo_bot_description)/urdf/inertia_macros.xacro" />
     <xacro:include filename="$(find mobo_bot_description)/urdf/robot_core.xacro" />

File: mobo_bot_description/urdf/sensors/sonar.xacro (robot description, xacro)
@@ -1,7 +1,4 @@
 <?xml version="1.0"?>
 <robot xmlns:xacro="http://www.ros.org/wiki/xacro">
-    <!-- <xacro:arg name="sonar_visual"   default="false"/> -->
-    <!-- <xacro:property name="deg2rad" value="0.017460317"/>
-    <xacro:property name="scan_angle" value="1"/> -->
     <xacro:macro name="insert_sonar" params="base_name parent_name x y z mass">
         <joint name="${base_name}_joint" type="fixed">
