Commit message: updated ign gz sim

File: mobo_bot_description/urdf/controllers/epmc_diff_drive_ros2_control.xacro (robot description, xacro)
@@ -1,5 +1,5 @@
 <?xml version="1.0"?>
 <robot xmlns:xacro="http://www.ros.org/wiki/xacro">
-    <ros2_control name="epmc_ros2_control" type="system">
+    <ros2_control name="epmc_diff_drive_ros2_control" type="system">
       <hardware>
         <plugin>epmc_hardware_interface/EPMCHardwareInterface</plugin>
@@ -11,6 +11,6 @@
       <joint name="left_wheel_joint">
         <command_interface name="velocity">
-            <param name="min">-8.0</param>
-            <param name="max">8.0</param>
+            <param name="min">-10.0</param>
+            <param name="max">10.0</param>
         </command_interface>
         <state_interface name="position"/>
@@ -19,6 +19,6 @@
       <joint name="right_wheel_joint">
         <command_interface name="velocity">
-            <param name="min">-8.0</param>
-            <param name="max">8.0</param>
+            <param name="min">-10.0</param>
+            <param name="max">10.0</param>
         </command_interface>
         <state_interface name="position"/>

File: mobo_bot_description/urdf/robot_core.xacro (robot description, xacro)
@@ -39,7 +39,5 @@
                 <cylinder radius="0.005" length="${chassis_height}"/>
             </geometry>
-            <material name="orange">
-                <color rgba="1 0.55 0 1"/>
-            </material>
+            <material name="orange"/>
         </visual>
         <visual>
@@ -48,7 +46,5 @@
                 <cylinder radius="0.005" length="${chassis_height}"/>
             </geometry>
-            <material name="orange">
-                <color rgba="1 0.55 0 1"/>
-            </material>
+            <material name="orange"/>
         </visual>
         <visual>
@@ -57,7 +53,5 @@
                 <cylinder radius="0.005" length="${chassis_height}"/>
             </geometry>
-            <material name="orange">
-                <color rgba="1 0.55 0 1"/>
-            </material>
+            <material name="orange"/>
         </visual>
         <visual>
@@ -66,7 +60,5 @@
                 <cylinder radius="0.005" length="${chassis_height}"/>
             </geometry>
-            <material name="orange">
-                <color rgba="1 0.55 0 1"/>
-            </material>
+            <material name="orange"/>
         </visual>
         <collision>
@@ -77,7 +69,14 @@
         </collision>
         <xacro:inertial_box mass="${chassis_mass}" x="${chassis_length}" y="${chassis_width}" z="${chassis_height}">
-            <origin xyz="-0.04 0 ${chassis_height/2}" rpy="0 0 0"/>
+            <origin xyz="-0.06 0 ${chassis_height/2}" rpy="0 0 0"/>
         </xacro:inertial_box>
     </link>
+    <xacro:if value="$(arg run_gz_sim)">
+        <gazebo reference="chassis">
+            <visual>
+              <xacro:gz_material_orange/>
+            </visual>
+        </gazebo>
+    </xacro:if>
     <xacro:insert_drive_wheel
         base_name="left_wheel"
@@ -87,6 +86,9 @@
         radius="${wheel_radius}"
         thickness="${wheel_width}"/>
-    <xacro:if value="$(arg use_simulation)">
+    <xacro:if value="$(arg run_gz_sim)">
         <gazebo reference="left_wheel">
+            <visual>
+              <xacro:gz_material_black/>
+            </visual>
             <mu1>1.0</mu1>
             <mu2>1.0</mu2>
@@ -99,4 +101,11 @@
         thickness="${wheel_width}"
         spoke_width="0.005"/>
+    <xacro:if value="$(arg run_gz_sim)">
+        <gazebo reference="left_rim">
+            <visual>
+              <xacro:gz_material_red/>
+            </visual>
+        </gazebo>
+    </xacro:if>
     <xacro:insert_drive_wheel
         base_name="right_wheel"
@@ -106,6 +115,9 @@
         radius="${wheel_radius}"
         thickness="${wheel_width}"/>
-    <xacro:if value="$(arg use_simulation)">
+    <xacro:if value="$(arg run_gz_sim)">
         <gazebo reference="right_wheel">
+            <visual>
+              <xacro:gz_material_black/>
+            </visual>
             <mu1>1.0</mu1>
             <mu2>1.0</mu2>
@@ -118,4 +130,11 @@
         thickness="${wheel_width}"
         spoke_width="0.005"/>
+    <xacro:if value="$(arg run_gz_sim)">
+        <gazebo reference="right_rim">
+            <visual>
+              <xacro:gz_material_red/>
+            </visual>
+        </gazebo>
+    </xacro:if>
     <joint name="castor_wheel_joint" type="fixed">
         <parent link="base_link"/>
@@ -143,6 +162,9 @@
         </xacro:inertial_sphere>
     </link>
-    <xacro:if value="$(arg use_simulation)">
+    <xacro:if value="$(arg run_gz_sim)">
         <gazebo reference="castor_wheel">
+            <visual>
+              <xacro:gz_material_silver/>
+            </visual>
             <mu1>0.001</mu1>
             <mu2>0.001</mu2>
@@ -155,26 +177,34 @@
         x="0.01" y="0" z="${chassis_height+lidar_z_offset}"
         mass="0.1"/>
-    <xacro:if value="$(arg use_simulation)">
+    <xacro:if value="$(arg run_gz_sim)">
       <gazebo reference="lidar">
+        <visual>
+          <xacro:gz_material_grey/>
+        </visual>
         <sensor name="lidar" type="gpu_lidar">
-          <pose> 0 0 0 0 0 0 </pose>
-          <ignition_frame_id>lidar</ignition_frame_id>
-          <topic>lidar/scan</topic>
+          <gz_frame_id>lidar</gz_frame_id>
+          <ray>
+            <scan>
+              <horizontal>
+                <samples>360</samples>
+                <min_angle>${-pi*2}</min_angle>
+                <max_angle>${pi*2}</max_angle>
+                <resolution>1</resolution>
+              </horizontal>
+            </scan>
+            <range>
+              <min>0.20</min>
+              <max>12.0</max>
+              <resolution>0.01</resolution>
+            </range>
+            <noise>
+              <type>gaussian</type>
+              <mean>0.0</mean>
+              <stddev>0.01</stddev>
+            </noise>
+          </ray>
           <always_on>true</always_on>
           <visualize>true</visualize>
-          <update_rate>10</update_rate>
-          <ray>
-            <scan>
-                <horizontal>
-                    <samples>360</samples>
-                    <min_angle>${-pi*2}</min_angle>
-                    <max_angle>${pi*2}</max_angle>
-                </horizontal>
-            </scan>
-            <range>
-                <min>0.1</min>
-                <max>10.0</max>
-            </range>
-          </ray>
+          <update_rate>10.0</update_rate>
         </sensor>
       </gazebo>
@@ -184,5 +214,5 @@
         parent_name="chassis"
         x="0" y="0" z="${chassis_height}"/>
-    <xacro:if value="$(arg use_simulation)">
+    <!-- <xacro:if value="$(arg run_gz_sim)">
           <gazebo reference="imu">
             <sensor name="imu" type="imu">
@@ -250,5 +280,5 @@
             </sensor>
         </gazebo>
-    </xacro:if>
+    </xacro:if> -->
     <xacro:insert_sonar
         base_name="sonar"
@@ -256,4 +286,11 @@
         x="0.0825" y="0" z="${chassis_height/6}"
         mass="0.005"/>
+    <xacro:if value="$(arg run_gz_sim)">
+        <gazebo reference="sonar">
+            <visual>
+              <xacro:gz_material_blue/>
+            </visual>
+        </gazebo>
+    </xacro:if>
     <xacro:property name="cam_x_offset" value="0.015"/>
     <xacro:property name="cam_z_offset" value="0.01"/>
@@ -263,13 +300,16 @@
         x="${0.08+cam_x_offset}" y="0" z="${chassis_height}"
         mass="0.005" tilt_angle="0.00"/>
-    <xacro:if value="$(arg use_simulation)">
-        <gazebo reference="camera_optical">
-          <sensor name="camera" type="camera">
-            <ignition_frame_id>camera_optical</ignition_frame_id>
+    <xacro:if value="$(arg run_gz_sim)">
+        <gazebo reference="camera">
+          <visual>
+            <xacro:gz_material_grey/>
+          </visual>
+          <sensor name="camera_optical" type="camera">
+            <gz_frame_id>camera</gz_frame_id>
             <camera>
               <horizontal_fov>1.047</horizontal_fov>
               <image>
-                <width>320</width>
-                <height>240</height>
+                <width>640</width>
+                <height>360</height>
               </image>
               <clip>
@@ -281,5 +321,5 @@
             <update_rate>30</update_rate>
             <visualize>true</visualize>
-            <topic>camera</topic>
+            <!-- <topic>camera</topic> -->
             <enable_metrics>true</enable_metrics>
           </sensor>

File: mobo_bot_description/urdf/robot_urdf.xacro (robot description, xacro)
@@ -1,12 +1,13 @@
 <?xml version="1.0"?>
 <robot name="mobo_bot" xmlns:xacro="http://www.ros.org/wiki/xacro">
-    <xacro:arg name="use_simulation" default="false"/>
+    <xacro:arg name="run_gz_sim" default="false"/>
+    <xacro:include filename="$(find mobo_bot_description)/urdf/color_macros.xacro" />
     <xacro:include filename="$(find mobo_bot_description)/urdf/inertia_macros.xacro" />
     <xacro:include filename="$(find mobo_bot_description)/urdf/robot_core.xacro" />
-    <xacro:if value="$(arg use_simulation)">
-        <xacro:include filename="$(find mobo_bot_description)/urdf/controllers/gazebo_control.xacro" />
+    <xacro:if value="$(arg run_gz_sim)">
+        <xacro:include filename="$(find mobo_bot_description)/urdf/controllers/gazebo_diff_drive_control.xacro" />
     </xacro:if>
-    <xacro:unless value="$(arg use_simulation)">
-        <xacro:include filename="$(find mobo_bot_description)/urdf/controllers/epmc_ros2_control.xacro" />
+    <xacro:unless value="$(arg run_gz_sim)">
+        <xacro:include filename="$(find mobo_bot_description)/urdf/controllers/epmc_diff_drive_ros2_control.xacro" />
     </xacro:unless>
 </robot>
